File: .history/02_POWER_24V_5V.kicad_sch (KiCad schematic)
At the start: 10 parts, among them U17 LMR51430

Commit message: 112
Parts:
- added COUT3: 100 µF, Capacitor_SMD:C_1210_3225Metric, symbol Device:C
- added RFBB1_TRIM1, RFBT1_TRIM1: DNP, Resistor_SMD:R_0805_2012Metric, symbol Device:R
- CIN1, CIN2, CIN3, COUT1, COUT2: footprint Capacitor_SMD:C_0805_2012Metric -> Capacitor_SMD:C_1210_3225Metric
- RFBB1: value 13.7k -> 15k
- RFBT1: value 100k -> 75k
- U31: renamed from U17; footprint Package_TO_SOT_SMD:SOT-23-6 -> my_footprints:SOT-23-THIN-6_DDC_TEX
- renumbered C9 to C35
Connections:
- net LOGIC_GND is gone; now on net GND: COUT1.2, COUT2.2, RFBB1.2
- net at RFBB1.1, RFBT1.2, U31.4 (FB): now also RFBB1_TRIM1.1, RFBT1_TRIM1.2
- net +5V renamed 5V_MAIN
- net 5V_MAIN: now also COUT3.1, RFBT1_TRIM1.1
- net FIELD_GND renamed GND
- net GND: now also COUT3.2, RFBB1_TRIM1.2

Commit message: 112
Parts:
- renumbered C35 to C32, U31 to U29
Changed lines of the file:
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@@
 		(dnp no)
 		(fields_autoplaced yes)
-		(property "Reference" "C35"
+		(property "Reference" "C32"
 			(at 128.27 40.64 90)
 			(show_name no)
@@
 			(project "MY_POWERFULL_PLC_PCB"
 				(path "/69a480d6-fa06-4fdd-8ed7-9beeb2ac027a/07a9e096-29cf-491a-9eb0-699b02d84850"
-					(reference "C35")
+					(reference "C32")
 					(unit 1)
 				)
@@
 		(in_pos_files yes)
 		(dnp no)
-		(property "Reference" "#PWR098"
+		(property "Reference" "#PWR099"
 			(at 62.23 62.23 0)
 			(hide yes)
@@
 			(project "MY_POWERFULL_PLC_PCB"
 				(path "/69a480d6-fa06-4fdd-8ed7-9beeb2ac027a/07a9e096-29cf-491a-9eb0-699b02d84850"
-					(reference "#PWR098")
+					(reference "#PWR099")
 					(unit 1)
 				)
@@
 		(in_pos_files yes)
 		(dnp no)
-		(property "Reference" "#PWR099"
+		(property "Reference" "#PWR0100"
 			(at 77.47 62.23 0)
 			(hide yes)
@@
 			(project "MY_POWERFULL_PLC_PCB"
 				(path "/69a480d6-fa06-4fdd-8ed7-9beeb2ac027a/07a9e096-29cf-491a-9eb0-699b02d84850"
-					(reference "#PWR099")
+					(reference "#PWR0100")
 					(unit 1)
 				)
@@
 		(in_pos_files yes)
 		(dnp no)
-		(property "Reference" "#PWR0100"
+		(property "Reference" "#PWR0101"
 			(at 90.17 62.23 0)
 			(hide yes)
@@
 			(project "MY_POWERFULL_PLC_PCB"
 				(path "/69a480d6-fa06-4fdd-8ed7-9beeb2ac027a/07a9e096-29cf-491a-9eb0-699b02d84850"
-					(reference "#PWR0100")
+					(reference "#PWR0101")
 					(unit 1)
 				)
@@
 		(in_pos_files yes)
 		(dnp no)
-		(property "Reference" "#PWR0103"
+		(property "Reference" "#PWR0104"
 			(at 156.21 46.99 0)
 			(hide yes)
@@
 			(project "MY_POWERFULL_PLC_PCB"
 				(path "/69a480d6-fa06-4fdd-8ed7-9beeb2ac027a/07a9e096-29cf-491a-9eb0-699b02d84850"
-					(reference "#PWR0103")
+					(reference "#PWR0104")
 					(unit 1)
 				)
@@
 		(in_pos_files yes)
 		(dnp no)
-		(property "Reference" "#PWR0102"
+		(property "Reference" "#PWR0103"
 			(at 147.32 72.39 0)
 			(hide yes)
@@
 			(project "MY_POWERFULL_PLC_PCB"
 				(path "/69a480d6-fa06-4fdd-8ed7-9beeb2ac027a/07a9e096-29cf-491a-9eb0-699b02d84850"
-					(reference "#PWR0102")
+					(reference "#PWR0103")
 					(unit 1)
 				)
@@
 		(in_pos_files yes)
 		(dnp no)
-		(property "Reference" "#PWR0101"
+		(property "Reference" "#PWR0102"
 			(at 114.3 64.77 0)
 			(hide yes)
@@
 			(project "MY_POWERFULL_PLC_PCB"
 				(path "/69a480d6-fa06-4fdd-8ed7-9beeb2ac027a/07a9e096-29cf-491a-9eb0-699b02d84850"
-					(reference "#PWR0101")
+					(reference "#PWR0102")
 					(unit 1)
 				)
@@
 		(in_pos_files yes)
 		(dnp no)
-		(property "Reference" "#PWR0106"
+		(property "Reference" "#PWR0107"
 			(at 187.96 46.99 0)
 			(hide yes)
@@
 			(project "MY_POWERFULL_PLC_PCB"
 				(path "/69a480d6-fa06-4fdd-8ed7-9beeb2ac027a/07a9e096-29cf-491a-9eb0-699b02d84850"
-					(reference "#PWR0106")
+					(reference "#PWR0107")
 					(unit 1)
 				)
@@
 		(in_pos_files yes)
 		(dnp no)
-		(property "Reference" "#PWR0104"
+		(property "Reference" "#PWR0105"
 			(at 158.75 72.39 0)
 			(hide yes)
@@
 			(project "MY_POWERFULL_PLC_PCB"
 				(path "/69a480d6-fa06-4fdd-8ed7-9beeb2ac027a/07a9e096-29cf-491a-9eb0-699b02d84850"
-					(reference "#PWR0104")
+					(reference "#PWR0105")
 					(unit 1)
 				)
@@
 		(dnp no)
 		(fields_autoplaced yes)
-		(property "Reference" "U31"
+		(property "Reference" "U29"
 			(at 114.3 40.64 0)
 			(show_name no)
@@
 			(project "MY_POWERFULL_PLC_PCB"
 				(path "/69a480d6-fa06-4fdd-8ed7-9beeb2ac027a/07a9e096-29cf-491a-9eb0-699b02d84850"
-					(reference "U31")
+					(reference "U29")
 					(unit 1)
 				)
@@
 		(dnp no)
 		(fields_autoplaced yes)
-		(property "Reference" "#PWR0107"
+		(property "Reference" "#PWR0108"
 			(at 201.93 53.34 0)
 			(hide yes)
@@
 			(project "MY_POWERFULL_PLC_PCB"
 				(path "/69a480d6-fa06-4fdd-8ed7-9beeb2ac027a/07a9e096-29cf-491a-9eb0-699b02d84850"
-					(reference "#PWR0107")
+					(reference "#PWR0108")
 					(unit 1)
 				)
@@
 		(in_pos_files yes)
 		(dnp no)
-		(property "Reference" "#PWR0105"
+		(property "Reference" "#PWR0106"
 			(at 171.45 46.99 0)
 			(hide yes)
@@
 			(project "MY_POWERFULL_PLC_PCB"
 				(path "/69a480d6-fa06-4fdd-8ed7-9beeb2ac027a/07a9e096-29cf-491a-9eb0-699b02d84850"
-					(reference "#PWR0105")
-					(unit 1)
-				)
+					(reference "#PWR0106")
+					(unit 1)
+				)

Commit message: 112
Connections:
- net 5V_MAIN renamed +5V
- net GND renamed Logic_GND
- net Logic_GND: no longer CIN1.2, CIN2.2, CIN3.2, U29.1 (GND)
- new net FIELD_GND: CIN1.2, CIN2.2, CIN3.2, U29.1 (GND)
Changed lines of the file:
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@@
 		(in_pos_files yes)
 		(dnp no)
-		(property "Reference" "#PWR098"
+		(property "Reference" "#PWR0156"
 			(at 62.23 62.23 0)
 			(hide yes)
@@
 			)
 		)
-		(property "Value" "GND"
+		(property "Value" "FIELD_GND"
 			(at 62.23 60.96 0)
 			(show_name no)
@@
 			(project "MY_POWERFULL_PLC_PCB"
 				(path "/69a480d6-fa06-4fdd-8ed7-9beeb2ac027a/07a9e096-29cf-491a-9eb0-699b02d84850"
-					(reference "#PWR098")
+					(reference "#PWR0156")
 					(unit 1)
 				)
@@
 		(in_pos_files yes)
 		(dnp no)
-		(property "Reference" "#PWR099"
+		(property "Reference" "#PWR0157"
 			(at 77.47 62.23 0)
 			(hide yes)
@@
 			)
 		)
-		(property "Value" "GND"
+		(property "Value" "FIELD_GND"
 			(at 77.47 60.96 0)
 			(show_name no)
@@
 			(project "MY_POWERFULL_PLC_PCB"
 				(path "/69a480d6-fa06-4fdd-8ed7-9beeb2ac027a/07a9e096-29cf-491a-9eb0-699b02d84850"
-					(reference "#PWR099")
+					(reference "#PWR0157")
 					(unit 1)
 				)
@@
 		(in_pos_files yes)
 		(dnp no)
-		(property "Reference" "#PWR0100"
+		(property "Reference" "#PWR0158"
 			(at 90.17 62.23 0)
 			(hide yes)
@@
 			)
 		)
-		(property "Value" "GND"
+		(property "Value" "FIELD_GND"
 			(at 90.17 60.96 0)
 			(show_name no)
@@
 			(project "MY_POWERFULL_PLC_PCB"
 				(path "/69a480d6-fa06-4fdd-8ed7-9beeb2ac027a/07a9e096-29cf-491a-9eb0-699b02d84850"
-					(reference "#PWR0100")
+					(reference "#PWR0158")
 					(unit 1)
 				)
@@
 		(in_pos_files yes)
 		(dnp no)
-		(property "Reference" "#PWR0103"
+		(property "Reference" "#PWR0161"
 			(at 156.21 46.99 0)
 			(hide yes)
@@
 			)
 		)
-		(property "Value" "GND"
+		(property "Value" "Logic_GND"
 			(at 156.21 45.72 0)
 			(show_name no)
@@
 			(project "MY_POWERFULL_PLC_PCB"
 				(path "/69a480d6-fa06-4fdd-8ed7-9beeb2ac027a/07a9e096-29cf-491a-9eb0-699b02d84850"
-					(reference "#PWR0103")
+					(reference "#PWR0161")
 					(unit 1)
 				)
@@
 		(in_pos_files yes)
 		(dnp no)
-		(property "Reference" "#PWR0102"
+		(property "Reference" "#PWR0160"
 			(at 147.32 72.39 0)
 			(hide yes)
@@
 			)
 		)
-		(property "Value" "GND"
+		(property "Value" "Logic_GND"
 			(at 147.32 71.12 0)
 			(show_name no)
@@
 			(project "MY_POWERFULL_PLC_PCB"
 				(path "/69a480d6-fa06-4fdd-8ed7-9beeb2ac027a/07a9e096-29cf-491a-9eb0-699b02d84850"
-					(reference "#PWR0102")
+					(reference "#PWR0160")
 					(unit 1)
 				)
@@
 		(in_pos_files yes)
 		(dnp no)
-		(property "Reference" "#PWR0101"
+		(property "Reference" "#PWR0159"
 			(at 114.3 64.77 0)
 			(hide yes)
@@
 			)
 		)
-		(property "Value" "GND"
+		(property "Value" "FIELD_GND"
 			(at 114.3 63.5 0)
 			(show_name no)
@@
 			(project "MY_POWERFULL_PLC_PCB"
 				(path "/69a480d6-fa06-4fdd-8ed7-9beeb2ac027a/07a9e096-29cf-491a-9eb0-699b02d84850"
-					(reference "#PWR0101")
+					(reference "#PWR0159")
 					(unit 1)
 				)
@@
 		(in_pos_files yes)
 		(dnp no)
-		(property "Reference" "#PWR0106"
+		(property "Reference" "#PWR0164"
 			(at 187.96 46.99 0)
 			(hide yes)
@@
 			)
 		)
-		(property "Value" "GND"
+		(property "Value" "Logic_GND"
 			(at 187.96 45.72 0)
 			(show_name no)
@@
 			(project "MY_POWERFULL_PLC_PCB"
 				(path "/69a480d6-fa06-4fdd-8ed7-9beeb2ac027a/07a9e096-29cf-491a-9eb0-699b02d84850"
-					(reference "#PWR0106")
+					(reference "#PWR0164")
 					(unit 1)
 				)
@@
 		(in_pos_files yes)
 		(dnp no)
-		(property "Reference" "#PWR0104"
+		(property "Reference" "#PWR0162"
 			(at 158.75 72.39 0)
 			(hide yes)
@@
 			)
 		)
-		(property "Value" "GND"
+		(property "Value" "Logic_GND"
 			(at 158.75 71.12 0)
 			(show_name no)
@@
 			(project "MY_POWERFULL_PLC_PCB"
 				(path "/69a480d6-fa06-4fdd-8ed7-9beeb2ac027a/07a9e096-29cf-491a-9eb0-699b02d84850"
-					(reference "#PWR0104")
+					(reference "#PWR0162")
 					(unit 1)
 				)
@@
 		(dnp no)
 		(fields_autoplaced yes)
-		(property "Reference" "#PWR0107"
+		(property "Reference" "#PWR0165"
 			(at 201.93 53.34 0)
 			(hide yes)
@@
 			)
 		)
-		(property "Value" "5V_MAIN"
+		(property "Value" "+5V"
 			(at 201.93 44.45 0)
 			(show_name no)
@@
 			(project "MY_POWERFULL_PLC_PCB"
 				(path "/69a480d6-fa06-4fdd-8ed7-9beeb2ac027a/07a9e096-29cf-491a-9eb0-699b02d84850"
-					(reference "#PWR0107")
+					(reference "#PWR0165")
 					(unit 1)
 				)
@@
 		(in_pos_files yes)
 		(dnp no)
-		(property "Reference" "#PWR0105"
+		(property "Reference" "#PWR0163"
 			(at 171.45 46.99 0)
 			(hide yes)
@@
 			)
 		)
-		(property "Value" "GND"
+		(property "Value" "Logic_GND"
 			(at 171.45 45.72 0)
 			(show_name no)
@@
 			(project "MY_POWERFULL_PLC_PCB"
 				(path "/69a480d6-fa06-4fdd-8ed7-9beeb2ac027a/07a9e096-29cf-491a-9eb0-699b02d84850"
-					(reference "#PWR0105")
-					(unit 1)
-				)
+					(reference "#PWR0163")
+					(unit 1)
+				)

Commit message: 112
Connections:
- net Logic_GND is gone; now on net FIELD_GND: COUT1.2, COUT2.2, COUT3.2, RFBB1.2, RFBB1_TRIM1.2
Changed lines of the file:
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@@
 		(in_pos_files yes)
 		(dnp no)
-		(property "Reference" "#PWR0156"
+		(property "Reference" "#PWR0148"
 			(at 62.23 62.23 0)
 			(hide yes)
@@
 			(project "MY_POWERFULL_PLC_PCB"
 				(path "/69a480d6-fa06-4fdd-8ed7-9beeb2ac027a/07a9e096-29cf-491a-9eb0-699b02d84850"
-					(reference "#PWR0156")
+					(reference "#PWR0148")
 					(unit 1)
 				)
@@
 		(in_pos_files yes)
 		(dnp no)
-		(property "Reference" "#PWR0157"
+		(property "Reference" "#PWR0149"
 			(at 77.47 62.23 0)
 			(hide yes)
@@
 			(project "MY_POWERFULL_PLC_PCB"
 				(path "/69a480d6-fa06-4fdd-8ed7-9beeb2ac027a/07a9e096-29cf-491a-9eb0-699b02d84850"
-					(reference "#PWR0157")
+					(reference "#PWR0149")
 					(unit 1)
 				)
@@
 		(in_pos_files yes)
 		(dnp no)
-		(property "Reference" "#PWR0158"
+		(property "Reference" "#PWR0150"
 			(at 90.17 62.23 0)
 			(hide yes)
@@
 			(project "MY_POWERFULL_PLC_PCB"
 				(path "/69a480d6-fa06-4fdd-8ed7-9beeb2ac027a/07a9e096-29cf-491a-9eb0-699b02d84850"
-					(reference "#PWR0158")
+					(reference "#PWR0150")
 					(unit 1)
 				)
@@
 		(in_pos_files yes)
 		(dnp no)
-		(property "Reference" "#PWR0161"
+		(property "Reference" "#PWR0153"
 			(at 156.21 46.99 0)
 			(hide yes)
@@
 			)
 		)
-		(property "Value" "Logic_GND"
+		(property "Value" "FIELD_GND"
 			(at 156.21 45.72 0)
 			(show_name no)
@@
 			(project "MY_POWERFULL_PLC_PCB"
 				(path "/69a480d6-fa06-4fdd-8ed7-9beeb2ac027a/07a9e096-29cf-491a-9eb0-699b02d84850"
-					(reference "#PWR0161")
+					(reference "#PWR0153")
 					(unit 1)
 				)
@@
 		(in_pos_files yes)
 		(dnp no)
-		(property "Reference" "#PWR0160"
+		(property "Reference" "#PWR0152"
 			(at 147.32 72.39 0)
 			(hide yes)
@@
 			)
 		)
-		(property "Value" "Logic_GND"
+		(property "Value" "FIELD_GND"
 			(at 147.32 71.12 0)
 			(show_name no)
@@
 			(project "MY_POWERFULL_PLC_PCB"
 				(path "/69a480d6-fa06-4fdd-8ed7-9beeb2ac027a/07a9e096-29cf-491a-9eb0-699b02d84850"
-					(reference "#PWR0160")
+					(reference "#PWR0152")
 					(unit 1)
 				)
@@
 		(in_pos_files yes)
 		(dnp no)
-		(property "Reference" "#PWR0159"
+		(property "Reference" "#PWR0151"
 			(at 114.3 64.77 0)
 			(hide yes)
@@
 			(project "MY_POWERFULL_PLC_PCB"
 				(path "/69a480d6-fa06-4fdd-8ed7-9beeb2ac027a/07a9e096-29cf-491a-9eb0-699b02d84850"
-					(reference "#PWR0159")
+					(reference "#PWR0151")
 					(unit 1)
 				)
@@
 		(in_pos_files yes)
 		(dnp no)
-		(property "Reference" "#PWR0164"
+		(property "Reference" "#PWR0156"
 			(at 187.96 46.99 0)
 			(hide yes)
@@
 			)
 		)
-		(property "Value" "Logic_GND"
+		(property "Value" "FIELD_GND"
 			(at 187.96 45.72 0)
 			(show_name no)
@@
 			(project "MY_POWERFULL_PLC_PCB"
 				(path "/69a480d6-fa06-4fdd-8ed7-9beeb2ac027a/07a9e096-29cf-491a-9eb0-699b02d84850"
-					(reference "#PWR0164")
+					(reference "#PWR0156")
 					(unit 1)
 				)
@@
 		(in_pos_files yes)
 		(dnp no)
-		(property "Reference" "#PWR0162"
+		(property "Reference" "#PWR0154"
 			(at 158.75 72.39 0)
 			(hide yes)
@@
 			)
 		)
-		(property "Value" "Logic_GND"
+		(property "Value" "FIELD_GND"
 			(at 158.75 71.12 0)
 			(show_name no)
@@
 			(project "MY_POWERFULL_PLC_PCB"
 				(path "/69a480d6-fa06-4fdd-8ed7-9beeb2ac027a/07a9e096-29cf-491a-9eb0-699b02d84850"
-					(reference "#PWR0162")
+					(reference "#PWR0154")
 					(unit 1)
 				)
@@
 		(dnp no)
 		(fields_autoplaced yes)
-		(property "Reference" "#PWR0165"
+		(property "Reference" "#PWR0157"
 			(at 201.93 53.34 0)
 			(hide yes)
@@
 			(project "MY_POWERFULL_PLC_PCB"
 				(path "/69a480d6-fa06-4fdd-8ed7-9beeb2ac027a/07a9e096-29cf-491a-9eb0-699b02d84850"
-					(reference "#PWR0165")
+					(reference "#PWR0157")
 					(unit 1)
 				)
@@
 		(in_pos_files yes)
 		(dnp no)
-		(property "Reference" "#PWR0163"
+		(property "Reference" "#PWR0155"
 			(at 171.45 46.99 0)
 			(hide yes)
@@
 			)
 		)
-		(property "Value" "Logic_GND"
+		(property "Value" "FIELD_GND"
 			(at 171.45 45.72 0)
 			(show_name no)
@@
 			(project "MY_POWERFULL_PLC_PCB"
 				(path "/69a480d6-fa06-4fdd-8ed7-9beeb2ac027a/07a9e096-29cf-491a-9eb0-699b02d84850"
-					(reference "#PWR0163")
-					(unit 1)
-				)
+					(reference "#PWR0155")
+					(unit 1)
+				)
