File: .history/03_POWER_5V_3V3.kicad_sch (KiCad schematic)
At the start: 5 parts, among them U18 AP7361C-33E

Commit message: 112
Parts:
- renumbered U18 to U32
Connections:
- net +3.3V renamed 3V3_LOGIC
- net +5V renamed 5V_MAIN
- net LOGIC_GND renamed GND
Changed lines of the file:
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@@
 		(in_pos_files yes)
 		(dnp no)
-		(property "Reference" "#PWR090"
+		(property "Reference" "#PWR0112"
 			(at 162.56 87.63 0)
 			(hide yes)
@@
 			)
 		)
-		(property "Value" "LOGIC_GND"
+		(property "Value" "GND"
 			(at 162.56 86.36 0)
 			(show_name no)
@@
 			(project "MY_POWERFULL_PLC_PCB"
 				(path "/69a480d6-fa06-4fdd-8ed7-9beeb2ac027a/0b17cd48-1203-4a6a-86a8-14ec70b25aae"
-					(reference "#PWR090")
+					(reference "#PWR0112")
 					(unit 1)
 				)
@@
 		(in_pos_files yes)
 		(dnp no)
-		(property "Reference" "#PWR091"
+		(property "Reference" "#PWR0113"
 			(at 177.8 87.63 0)
 			(hide yes)
@@
 			)
 		)
-		(property "Value" "LOGIC_GND"
+		(property "Value" "GND"
 			(at 177.8 86.36 0)
 			(show_name no)
@@
 			(project "MY_POWERFULL_PLC_PCB"
 				(path "/69a480d6-fa06-4fdd-8ed7-9beeb2ac027a/0b17cd48-1203-4a6a-86a8-14ec70b25aae"
-					(reference "#PWR091")
+					(reference "#PWR0113")
 					(unit 1)
 				)
@@
 		(in_pos_files yes)
 		(dnp no)
-		(property "Reference" "#PWR088"
+		(property "Reference" "#PWR0110"
 			(at 132.08 87.63 0)
 			(hide yes)
@@
 			)
 		)
-		(property "Value" "LOGIC_GND"
+		(property "Value" "GND"
 			(at 132.08 86.36 0)
 			(show_name no)
@@
 			(project "MY_POWERFULL_PLC_PCB"
 				(path "/69a480d6-fa06-4fdd-8ed7-9beeb2ac027a/0b17cd48-1203-4a6a-86a8-14ec70b25aae"
-					(reference "#PWR088")
+					(reference "#PWR0110")
 					(unit 1)
 				)
@@
 		(dnp no)
 		(fields_autoplaced yes)
-		(property "Reference" "U18"
+		(property "Reference" "U32"
 			(at 151.13 67.31 0)
 			(show_name no)
@@
 			(project "MY_POWERFULL_PLC_PCB"
 				(path "/69a480d6-fa06-4fdd-8ed7-9beeb2ac027a/0b17cd48-1203-4a6a-86a8-14ec70b25aae"
-					(reference "U18")
+					(reference "U32")
 					(unit 1)
 				)
@@
 		(in_pos_files yes)
 		(dnp no)
-		(property "Reference" "#PWR089"
+		(property "Reference" "#PWR0111"
 			(at 151.13 87.63 0)
 			(hide yes)
@@
 			)
 		)
-		(property "Value" "LOGIC_GND"
+		(property "Value" "GND"
 			(at 151.13 86.36 0)
 			(show_name no)
@@
 			(project "MY_POWERFULL_PLC_PCB"
 				(path "/69a480d6-fa06-4fdd-8ed7-9beeb2ac027a/0b17cd48-1203-4a6a-86a8-14ec70b25aae"
-					(reference "#PWR089")
+					(reference "#PWR0111")
 					(unit 1)
 				)
@@
 		(dnp no)
 		(fields_autoplaced yes)
-		(property "Reference" "#PWR086"
+		(property "Reference" "#PWR0108"
 			(at 116.84 77.47 0)
 			(hide yes)
@@
 			)
 		)
-		(property "Value" "+5V"
+		(property "Value" "5V_MAIN"
 			(at 116.84 68.58 0)
 			(show_name no)
@@
 			(project "MY_POWERFULL_PLC_PCB"
 				(path "/69a480d6-fa06-4fdd-8ed7-9beeb2ac027a/0b17cd48-1203-4a6a-86a8-14ec70b25aae"
-					(reference "#PWR086")
+					(reference "#PWR0108")
 					(unit 1)
 				)
@@
 		(in_pos_files yes)
 		(dnp no)
-		(property "Reference" "#PWR087"
+		(property "Reference" "#PWR0109"
 			(at 120.65 87.63 0)
 			(hide yes)
@@
 			)
 		)
-		(property "Value" "LOGIC_GND"
+		(property "Value" "GND"
 			(at 120.65 86.36 0)
 			(show_name no)
@@
 			(project "MY_POWERFULL_PLC_PCB"
 				(path "/69a480d6-fa06-4fdd-8ed7-9beeb2ac027a/0b17cd48-1203-4a6a-86a8-14ec70b25aae"
-					(reference "#PWR087")
+					(reference "#PWR0109")
 					(unit 1)
 				)
@@
 		(dnp no)
 		(fields_autoplaced yes)
-		(property "Reference" "#PWR092"
+		(property "Reference" "#PWR0114"
 			(at 193.04 77.47 0)
 			(hide yes)
@@
 			)
 		)
-		(property "Value" "+3.3V"
+		(property "Value" "3V3_LOGIC"
 			(at 193.04 68.58 0)
 			(show_name no)
@@
 			(project "MY_POWERFULL_PLC_PCB"
 				(path "/69a480d6-fa06-4fdd-8ed7-9beeb2ac027a/0b17cd48-1203-4a6a-86a8-14ec70b25aae"
-					(reference "#PWR092")
-					(unit 1)
-				)
+					(reference "#PWR0114")
+					(unit 1)
+				)

Commit message: 112
Parts:
- renumbered U32 to U30
Changed lines of the file:
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@@
 		(in_pos_files yes)
 		(dnp no)
-		(property "Reference" "#PWR0112"
+		(property "Reference" "#PWR0113"
 			(at 162.56 87.63 0)
 			(hide yes)
@@
 			(project "MY_POWERFULL_PLC_PCB"
 				(path "/69a480d6-fa06-4fdd-8ed7-9beeb2ac027a/0b17cd48-1203-4a6a-86a8-14ec70b25aae"
-					(reference "#PWR0112")
+					(reference "#PWR0113")
 					(unit 1)
 				)
@@
 		(in_pos_files yes)
 		(dnp no)
-		(property "Reference" "#PWR0113"
+		(property "Reference" "#PWR0114"
 			(at 177.8 87.63 0)
 			(hide yes)
@@
 			(project "MY_POWERFULL_PLC_PCB"
 				(path "/69a480d6-fa06-4fdd-8ed7-9beeb2ac027a/0b17cd48-1203-4a6a-86a8-14ec70b25aae"
-					(reference "#PWR0113")
+					(reference "#PWR0114")
 					(unit 1)
 				)
@@
 		(in_pos_files yes)
 		(dnp no)
-		(property "Reference" "#PWR0110"
+		(property "Reference" "#PWR0111"
 			(at 132.08 87.63 0)
 			(hide yes)
@@
 			(project "MY_POWERFULL_PLC_PCB"
 				(path "/69a480d6-fa06-4fdd-8ed7-9beeb2ac027a/0b17cd48-1203-4a6a-86a8-14ec70b25aae"
-					(reference "#PWR0110")
+					(reference "#PWR0111")
 					(unit 1)
 				)
@@
 		(dnp no)
 		(fields_autoplaced yes)
-		(property "Reference" "U32"
+		(property "Reference" "U30"
 			(at 151.13 67.31 0)
 			(show_name no)
@@
 			(project "MY_POWERFULL_PLC_PCB"
 				(path "/69a480d6-fa06-4fdd-8ed7-9beeb2ac027a/0b17cd48-1203-4a6a-86a8-14ec70b25aae"
-					(reference "U32")
+					(reference "U30")
 					(unit 1)
 				)
@@
 		(in_pos_files yes)
 		(dnp no)
-		(property "Reference" "#PWR0111"
+		(property "Reference" "#PWR0112"
 			(at 151.13 87.63 0)
 			(hide yes)
@@
 			(project "MY_POWERFULL_PLC_PCB"
 				(path "/69a480d6-fa06-4fdd-8ed7-9beeb2ac027a/0b17cd48-1203-4a6a-86a8-14ec70b25aae"
-					(reference "#PWR0111")
+					(reference "#PWR0112")
 					(unit 1)
 				)
@@
 		(dnp no)
 		(fields_autoplaced yes)
-		(property "Reference" "#PWR0108"
+		(property "Reference" "#PWR0109"
 			(at 116.84 77.47 0)
 			(hide yes)
@@
 			(project "MY_POWERFULL_PLC_PCB"
 				(path "/69a480d6-fa06-4fdd-8ed7-9beeb2ac027a/0b17cd48-1203-4a6a-86a8-14ec70b25aae"
-					(reference "#PWR0108")
+					(reference "#PWR0109")
 					(unit 1)
 				)
@@
 		(in_pos_files yes)
 		(dnp no)
-		(property "Reference" "#PWR0109"
+		(property "Reference" "#PWR0110"
 			(at 120.65 87.63 0)
 			(hide yes)
@@
 			(project "MY_POWERFULL_PLC_PCB"
 				(path "/69a480d6-fa06-4fdd-8ed7-9beeb2ac027a/0b17cd48-1203-4a6a-86a8-14ec70b25aae"
-					(reference "#PWR0109")
+					(reference "#PWR0110")
 					(unit 1)
 				)
@@
 		(dnp no)
 		(fields_autoplaced yes)
-		(property "Reference" "#PWR0114"
+		(property "Reference" "#PWR0115"
 			(at 193.04 77.47 0)
 			(hide yes)
@@
 			(project "MY_POWERFULL_PLC_PCB"
 				(path "/69a480d6-fa06-4fdd-8ed7-9beeb2ac027a/0b17cd48-1203-4a6a-86a8-14ec70b25aae"
-					(reference "#PWR0114")
-					(unit 1)
-				)
+					(reference "#PWR0115")
+					(unit 1)
+				)

Commit message: 112
Connections:
- net 3V3_LOGIC renamed +3V3
- net 5V_MAIN renamed +5V
- net GND renamed Logic_GND
Changed lines of the file:
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@@
 		(in_pos_files yes)
 		(dnp no)
-		(property "Reference" "#PWR0112"
+		(property "Reference" "#PWR0170"
 			(at 162.56 87.63 0)
 			(hide yes)
@@
 			)
 		)
-		(property "Value" "GND"
+		(property "Value" "Logic_GND"
 			(at 162.56 86.36 0)
 			(show_name no)
@@
 			(project "MY_POWERFULL_PLC_PCB"
 				(path "/69a480d6-fa06-4fdd-8ed7-9beeb2ac027a/0b17cd48-1203-4a6a-86a8-14ec70b25aae"
-					(reference "#PWR0112")
+					(reference "#PWR0170")
 					(unit 1)
 				)
@@
 		(in_pos_files yes)
 		(dnp no)
-		(property "Reference" "#PWR0113"
+		(property "Reference" "#PWR0171"
 			(at 177.8 87.63 0)
 			(hide yes)
@@
 			)
 		)
-		(property "Value" "GND"
+		(property "Value" "Logic_GND"
 			(at 177.8 86.36 0)
 			(show_name no)
@@
 			(project "MY_POWERFULL_PLC_PCB"
 				(path "/69a480d6-fa06-4fdd-8ed7-9beeb2ac027a/0b17cd48-1203-4a6a-86a8-14ec70b25aae"
-					(reference "#PWR0113")
+					(reference "#PWR0171")
 					(unit 1)
 				)
@@
 		(in_pos_files yes)
 		(dnp no)
-		(property "Reference" "#PWR0110"
+		(property "Reference" "#PWR0168"
 			(at 132.08 87.63 0)
 			(hide yes)
@@
 			)
 		)
-		(property "Value" "GND"
+		(property "Value" "Logic_GND"
 			(at 132.08 86.36 0)
 			(show_name no)
@@
 			(project "MY_POWERFULL_PLC_PCB"
 				(path "/69a480d6-fa06-4fdd-8ed7-9beeb2ac027a/0b17cd48-1203-4a6a-86a8-14ec70b25aae"
-					(reference "#PWR0110")
+					(reference "#PWR0168")
 					(unit 1)
 				)
@@
 		(in_pos_files yes)
 		(dnp no)
-		(property "Reference" "#PWR0111"
+		(property "Reference" "#PWR0169"
 			(at 151.13 87.63 0)
 			(hide yes)
@@
 			)
 		)
-		(property "Value" "GND"
+		(property "Value" "Logic_GND"
 			(at 151.13 86.36 0)
 			(show_name no)
@@
 			(project "MY_POWERFULL_PLC_PCB"
 				(path "/69a480d6-fa06-4fdd-8ed7-9beeb2ac027a/0b17cd48-1203-4a6a-86a8-14ec70b25aae"
-					(reference "#PWR0111")
+					(reference "#PWR0169")
 					(unit 1)
 				)
@@
 		(dnp no)
 		(fields_autoplaced yes)
-		(property "Reference" "#PWR0108"
+		(property "Reference" "#PWR0166"
 			(at 116.84 77.47 0)
 			(hide yes)
@@
 			)
 		)
-		(property "Value" "5V_MAIN"
+		(property "Value" "+5V"
 			(at 116.84 68.58 0)
 			(show_name no)
@@
 			(project "MY_POWERFULL_PLC_PCB"
 				(path "/69a480d6-fa06-4fdd-8ed7-9beeb2ac027a/0b17cd48-1203-4a6a-86a8-14ec70b25aae"
-					(reference "#PWR0108")
+					(reference "#PWR0166")
 					(unit 1)
 				)
@@
 		(in_pos_files yes)
 		(dnp no)
-		(property "Reference" "#PWR0109"
+		(property "Reference" "#PWR0167"
 			(at 120.65 87.63 0)
 			(hide yes)
@@
 			)
 		)
-		(property "Value" "GND"
+		(property "Value" "Logic_GND"
 			(at 120.65 86.36 0)
 			(show_name no)
@@
 			(project "MY_POWERFULL_PLC_PCB"
 				(path "/69a480d6-fa06-4fdd-8ed7-9beeb2ac027a/0b17cd48-1203-4a6a-86a8-14ec70b25aae"
-					(reference "#PWR0109")
+					(reference "#PWR0167")
 					(unit 1)
 				)
@@
 		(dnp no)
 		(fields_autoplaced yes)
-		(property "Reference" "#PWR0114"
+		(property "Reference" "#PWR0172"
 			(at 193.04 77.47 0)
 			(hide yes)
@@
 			)
 		)
-		(property "Value" "3V3_LOGIC"
+		(property "Value" "+3V3"
 			(at 193.04 68.58 0)
 			(show_name no)
@@
 			(project "MY_POWERFULL_PLC_PCB"
 				(path "/69a480d6-fa06-4fdd-8ed7-9beeb2ac027a/0b17cd48-1203-4a6a-86a8-14ec70b25aae"
-					(reference "#PWR0114")
-					(unit 1)
-				)
+					(reference "#PWR0172")
+					(unit 1)
+				)

Commit message: 112
Connections:
- net Logic_GND renamed FIELD_GND
Changed lines of the file:
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@@
 		(in_pos_files yes)
 		(dnp no)
-		(property "Reference" "#PWR0170"
+		(property "Reference" "#PWR0162"
 			(at 162.56 87.63 0)
 			(hide yes)
@@
 			)
 		)
-		(property "Value" "Logic_GND"
+		(property "Value" "FIELD_GND"
 			(at 162.56 86.36 0)
 			(show_name no)
@@
 			(project "MY_POWERFULL_PLC_PCB"
 				(path "/69a480d6-fa06-4fdd-8ed7-9beeb2ac027a/0b17cd48-1203-4a6a-86a8-14ec70b25aae"
-					(reference "#PWR0170")
+					(reference "#PWR0162")
 					(unit 1)
 				)
@@
 		(in_pos_files yes)
 		(dnp no)
-		(property "Reference" "#PWR0171"
+		(property "Reference" "#PWR0163"
 			(at 177.8 87.63 0)
 			(hide yes)
@@
 			)
 		)
-		(property "Value" "Logic_GND"
+		(property "Value" "FIELD_GND"
 			(at 177.8 86.36 0)
 			(show_name no)
@@
 			(project "MY_POWERFULL_PLC_PCB"
 				(path "/69a480d6-fa06-4fdd-8ed7-9beeb2ac027a/0b17cd48-1203-4a6a-86a8-14ec70b25aae"
-					(reference "#PWR0171")
+					(reference "#PWR0163")
 					(unit 1)
 				)
@@
 		(in_pos_files yes)
 		(dnp no)
-		(property "Reference" "#PWR0168"
+		(property "Reference" "#PWR0160"
 			(at 132.08 87.63 0)
 			(hide yes)
@@
 			)
 		)
-		(property "Value" "Logic_GND"
+		(property "Value" "FIELD_GND"
 			(at 132.08 86.36 0)
 			(show_name no)
@@
 			(project "MY_POWERFULL_PLC_PCB"
 				(path "/69a480d6-fa06-4fdd-8ed7-9beeb2ac027a/0b17cd48-1203-4a6a-86a8-14ec70b25aae"
-					(reference "#PWR0168")
+					(reference "#PWR0160")
 					(unit 1)
 				)
@@
 		(in_pos_files yes)
 		(dnp no)
-		(property "Reference" "#PWR0169"
+		(property "Reference" "#PWR0161"
 			(at 151.13 87.63 0)
 			(hide yes)
@@
 			)
 		)
-		(property "Value" "Logic_GND"
+		(property "Value" "FIELD_GND"
 			(at 151.13 86.36 0)
 			(show_name no)
@@
 			(project "MY_POWERFULL_PLC_PCB"
 				(path "/69a480d6-fa06-4fdd-8ed7-9beeb2ac027a/0b17cd48-1203-4a6a-86a8-14ec70b25aae"
-					(reference "#PWR0169")
+					(reference "#PWR0161")
 					(unit 1)
 				)
@@
 		(dnp no)
 		(fields_autoplaced yes)
-		(property "Reference" "#PWR0166"
+		(property "Reference" "#PWR0158"
 			(at 116.84 77.47 0)
 			(hide yes)
@@
 			(project "MY_POWERFULL_PLC_PCB"
 				(path "/69a480d6-fa06-4fdd-8ed7-9beeb2ac027a/0b17cd48-1203-4a6a-86a8-14ec70b25aae"
-					(reference "#PWR0166")
+					(reference "#PWR0158")
 					(unit 1)
 				)
@@
 		(in_pos_files yes)
 		(dnp no)
-		(property "Reference" "#PWR0167"
+		(property "Reference" "#PWR0159"
 			(at 120.65 87.63 0)
 			(hide yes)
@@
 			)
 		)
-		(property "Value" "Logic_GND"
+		(property "Value" "FIELD_GND"
 			(at 120.65 86.36 0)
 			(show_name no)
@@
 			(project "MY_POWERFULL_PLC_PCB"
 				(path "/69a480d6-fa06-4fdd-8ed7-9beeb2ac027a/0b17cd48-1203-4a6a-86a8-14ec70b25aae"
-					(reference "#PWR0167")
+					(reference "#PWR0159")
 					(unit 1)
 				)
@@
 		(dnp no)
 		(fields_autoplaced yes)
-		(property "Reference" "#PWR0172"
+		(property "Reference" "#PWR0164"
 			(at 193.04 77.47 0)
 			(hide yes)
@@
 			(project "MY_POWERFULL_PLC_PCB"
 				(path "/69a480d6-fa06-4fdd-8ed7-9beeb2ac027a/0b17cd48-1203-4a6a-86a8-14ec70b25aae"
-					(reference "#PWR0172")
-					(unit 1)
-				)
+					(reference "#PWR0164")
+					(unit 1)
+				)
