File: .history/DI_Fast_Module.kicad_sch (KiCad schematic)
At the start: 10 parts, among them U3 SN74LVC1G17DBVR, U4 6N137

Commit message: 112
Parts:
- renumbered U3 to U2, U4 to U3

Commit message: 112
Connections:
- net Field_GND renamed FIELD_GND
- net Logic_GND renamed LOGIC_GND

Commit message: 112
Connections:
- net LOGIC_GND renamed Logic_GND
