File: .history/DI_Module.kicad_sch (KiCad schematic)
At the start: 10 parts, among them U15 SN74LVC1G14DBV, U16 LTV-357T

Commit message: 112
Parts:
- renumbered C19 to C16, C20 to C17, D13 to D11, D14 to D12, R21 to R18, R22 to R19, R23 to R20, R24 to R21, U15 to U13, U16 to U14
