File: .history/DO_FAST.kicad_sch (KiCad schematic)
At the start: 8 parts, among them Q10 NMOS AOD4184A, U37 UCC27511ADBV

Commit message: 112
Parts:
- renumbered C42 to C36, C43 to C37, R75 to R69, R76 to R70, R77 to R71, R78 to R72, U37 to U33

Commit message: 112
Parts:
- Q10: footprint Package_TO_SOT_THT:TO-220-3_Vertical -> Package_TO_SOT_SMD:TO-252-3_TabPin2
Changed lines of the file:
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@@
 		(in_pos_files yes)
 		(dnp no)
-		(property "Reference" "#PWR0150"
+		(property "Reference" "#PWR0149"
 			(at 96.52 57.15 0)
 			(hide yes)
@@
 			(project "MY_POWERFULL_PLC_PCB"
 				(path "/69a480d6-fa06-4fdd-8ed7-9beeb2ac027a/ea39046e-ca02-46d1-9fd4-b85a58c0b80f/4e719e6a-f498-4860-85c2-d3c910fb7d70"
-					(reference "#PWR0150")
+					(reference "#PWR0149")
 					(unit 1)
 				)
 				(path "/69a480d6-fa06-4fdd-8ed7-9beeb2ac027a/ea39046e-ca02-46d1-9fd4-b85a58c0b80f/5918cb53-767b-4406-8a2b-be52ced64ae0"
-					(reference "#PWR0170")
+					(reference "#PWR0169")
 					(unit 1)
 				)
 				(path "/69a480d6-fa06-4fdd-8ed7-9beeb2ac027a/ea39046e-ca02-46d1-9fd4-b85a58c0b80f/6ec847d1-af3b-47e2-b394-844cce0f53eb"
-					(reference "#PWR0165")
+					(reference "#PWR0164")
 					(unit 1)
 				)
 				(path "/69a480d6-fa06-4fdd-8ed7-9beeb2ac027a/ea39046e-ca02-46d1-9fd4-b85a58c0b80f/938b05e1-ee13-4e84-85e5-d171a1a5f239"
-					(reference "#PWR0185")
+					(reference "#PWR0184")
 					(unit 1)
 				)
 				(path "/69a480d6-fa06-4fdd-8ed7-9beeb2ac027a/ea39046e-ca02-46d1-9fd4-b85a58c0b80f/94887116-e992-4614-87b1-1893944a34af"
-					(reference "#PWR0180")
+					(reference "#PWR0179")
 					(unit 1)
 				)
 				(path "/69a480d6-fa06-4fdd-8ed7-9beeb2ac027a/ea39046e-ca02-46d1-9fd4-b85a58c0b80f/976e15ae-69f2-46a4-92b9-157eb83b98b3"
-					(reference "#PWR0175")
+					(reference "#PWR0174")
 					(unit 1)
 				)
 				(path "/69a480d6-fa06-4fdd-8ed7-9beeb2ac027a/ea39046e-ca02-46d1-9fd4-b85a58c0b80f/9dcca28d-a41c-4e95-8119-28bf2da75604"
-					(reference "#PWR0160")
+					(reference "#PWR0159")
 					(unit 1)
 				)
 				(path "/69a480d6-fa06-4fdd-8ed7-9beeb2ac027a/ea39046e-ca02-46d1-9fd4-b85a58c0b80f/bdb5a479-48da-432b-97a9-55765e4484ff"
-					(reference "#PWR0155")
+					(reference "#PWR0154")
 					(unit 1)
 				)
@@
 		(in_pos_files yes)
 		(dnp no)
-		(property "Reference" "#PWR0148"
+		(property "Reference" "#PWR0147"
 			(at 54.61 96.52 0)
 			(hide yes)
@@
 			(project "MY_POWERFULL_PLC_PCB"
 				(path "/69a480d6-fa06-4fdd-8ed7-9beeb2ac027a/ea39046e-ca02-46d1-9fd4-b85a58c0b80f/4e719e6a-f498-4860-85c2-d3c910fb7d70"
-					(reference "#PWR0148")
+					(reference "#PWR0147")
 					(unit 1)
 				)
 				(path "/69a480d6-fa06-4fdd-8ed7-9beeb2ac027a/ea39046e-ca02-46d1-9fd4-b85a58c0b80f/5918cb53-767b-4406-8a2b-be52ced64ae0"
-					(reference "#PWR0168")
+					(reference "#PWR0167")
 					(unit 1)
 				)
 				(path "/69a480d6-fa06-4fdd-8ed7-9beeb2ac027a/ea39046e-ca02-46d1-9fd4-b85a58c0b80f/6ec847d1-af3b-47e2-b394-844cce0f53eb"
-					(reference "#PWR0163")
+					(reference "#PWR0162")
 					(unit 1)
 				)
 				(path "/69a480d6-fa06-4fdd-8ed7-9beeb2ac027a/ea39046e-ca02-46d1-9fd4-b85a58c0b80f/938b05e1-ee13-4e84-85e5-d171a1a5f239"
-					(reference "#PWR0183")
+					(reference "#PWR0182")
 					(unit 1)
 				)
 				(path "/69a480d6-fa06-4fdd-8ed7-9beeb2ac027a/ea39046e-ca02-46d1-9fd4-b85a58c0b80f/94887116-e992-4614-87b1-1893944a34af"
-					(reference "#PWR0178")
+					(reference "#PWR0177")
 					(unit 1)
 				)
 				(path "/69a480d6-fa06-4fdd-8ed7-9beeb2ac027a/ea39046e-ca02-46d1-9fd4-b85a58c0b80f/976e15ae-69f2-46a4-92b9-157eb83b98b3"
-					(reference "#PWR0173")
+					(reference "#PWR0172")
 					(unit 1)
 				)
 				(path "/69a480d6-fa06-4fdd-8ed7-9beeb2ac027a/ea39046e-ca02-46d1-9fd4-b85a58c0b80f/9dcca28d-a41c-4e95-8119-28bf2da75604"
-					(reference "#PWR0158")
+					(reference "#PWR0157")
 					(unit 1)
 				)
 				(path "/69a480d6-fa06-4fdd-8ed7-9beeb2ac027a/ea39046e-ca02-46d1-9fd4-b85a58c0b80f/bdb5a479-48da-432b-97a9-55765e4484ff"
-					(reference "#PWR0153")
+					(reference "#PWR0152")
 					(unit 1)
 				)
@@
 		(in_pos_files yes)
 		(dnp no)
-		(property "Reference" "#PWR0149"
+		(property "Reference" "#PWR0148"
 			(at 59.69 52.07 0)
 			(hide yes)
@@
 			(project "MY_POWERFULL_PLC_PCB"
 				(path "/69a480d6-fa06-4fdd-8ed7-9beeb2ac027a/ea39046e-ca02-46d1-9fd4-b85a58c0b80f/4e719e6a-f498-4860-85c2-d3c910fb7d70"
-					(reference "#PWR0149")
+					(reference "#PWR0148")
 					(unit 1)
 				)
 				(path "/69a480d6-fa06-4fdd-8ed7-9beeb2ac027a/ea39046e-ca02-46d1-9fd4-b85a58c0b80f/5918cb53-767b-4406-8a2b-be52ced64ae0"
-					(reference "#PWR0169")
+					(reference "#PWR0168")
 					(unit 1)
 				)
 				(path "/69a480d6-fa06-4fdd-8ed7-9beeb2ac027a/ea39046e-ca02-46d1-9fd4-b85a58c0b80f/6ec847d1-af3b-47e2-b394-844cce0f53eb"
-					(reference "#PWR0164")
+					(reference "#PWR0163")
 					(unit 1)
 				)
 				(path "/69a480d6-fa06-4fdd-8ed7-9beeb2ac027a/ea39046e-ca02-46d1-9fd4-b85a58c0b80f/938b05e1-ee13-4e84-85e5-d171a1a5f239"
-					(reference "#PWR0184")
+					(reference "#PWR0183")
 					(unit 1)
 				)
 				(path "/69a480d6-fa06-4fdd-8ed7-9beeb2ac027a/ea39046e-ca02-46d1-9fd4-b85a58c0b80f/94887116-e992-4614-87b1-1893944a34af"
-					(reference "#PWR0179")
+					(reference "#PWR0178")
 					(unit 1)
 				)
 				(path "/69a480d6-fa06-4fdd-8ed7-9beeb2ac027a/ea39046e-ca02-46d1-9fd4-b85a58c0b80f/976e15ae-69f2-46a4-92b9-157eb83b98b3"
-					(reference "#PWR0174")
+					(reference "#PWR0173")
 					(unit 1)
 				)
 				(path "/69a480d6-fa06-4fdd-8ed7-9beeb2ac027a/ea39046e-ca02-46d1-9fd4-b85a58c0b80f/9dcca28d-a41c-4e95-8119-28bf2da75604"
-					(reference "#PWR0159")
+					(reference "#PWR0158")
 					(unit 1)
 				)
 				(path "/69a480d6-fa06-4fdd-8ed7-9beeb2ac027a/ea39046e-ca02-46d1-9fd4-b85a58c0b80f/bdb5a479-48da-432b-97a9-55765e4484ff"
-					(reference "#PWR0154")
+					(reference "#PWR0153")
 					(unit 1)
 				)
@@
 		(dnp no)
 		(fields_autoplaced yes)
-		(property "Reference" "#PWR0147"
+		(property "Reference" "#PWR0146"
 			(at 54.61 83.82 0)
 			(hide yes)
@@
 			(project "MY_POWERFULL_PLC_PCB"
 				(path "/69a480d6-fa06-4fdd-8ed7-9beeb2ac027a/ea39046e-ca02-46d1-9fd4-b85a58c0b80f/4e719e6a-f498-4860-85c2-d3c910fb7d70"
-					(reference "#PWR0147")
+					(reference "#PWR0146")
 					(unit 1)
 				)
 				(path "/69a480d6-fa06-4fdd-8ed7-9beeb2ac027a/ea39046e-ca02-46d1-9fd4-b85a58c0b80f/5918cb53-767b-4406-8a2b-be52ced64ae0"
-					(reference "#PWR0167")
+					(reference "#PWR0166")
 					(unit 1)
 				)
 				(path "/69a480d6-fa06-4fdd-8ed7-9beeb2ac027a/ea39046e-ca02-46d1-9fd4-b85a58c0b80f/6ec847d1-af3b-47e2-b394-844cce0f53eb"
-					(reference "#PWR0162")
+					(reference "#PWR0161")
 					(unit 1)
 				)
 				(path "/69a480d6-fa06-4fdd-8ed7-9beeb2ac027a/ea39046e-ca02-46d1-9fd4-b85a58c0b80f/938b05e1-ee13-4e84-85e5-d171a1a5f239"
-					(reference "#PWR0182")
+					(reference "#PWR0181")
 					(unit 1)
 				)
 				(path "/69a480d6-fa06-4fdd-8ed7-9beeb2ac027a/ea39046e-ca02-46d1-9fd4-b85a58c0b80f/94887116-e992-4614-87b1-1893944a34af"
-					(reference "#PWR0177")
+					(reference "#PWR0176")
 					(unit 1)
 				)
 				(path "/69a480d6-fa06-4fdd-8ed7-9beeb2ac027a/ea39046e-ca02-46d1-9fd4-b85a58c0b80f/976e15ae-69f2-46a4-92b9-157eb83b98b3"
-					(reference "#PWR0172")
+					(reference "#PWR0171")
 					(unit 1)
 				)
 				(path "/69a480d6-fa06-4fdd-8ed7-9beeb2ac027a/ea39046e-ca02-46d1-9fd4-b85a58c0b80f/9dcca28d-a41c-4e95-8119-28bf2da75604"
-					(reference "#PWR0157")
+					(reference "#PWR0156")
 					(unit 1)
 				)
 				(path "/69a480d6-fa06-4fdd-8ed7-9beeb2ac027a/ea39046e-ca02-46d1-9fd4-b85a58c0b80f/bdb5a479-48da-432b-97a9-55765e4484ff"
-					(reference "#PWR0152")
+					(reference "#PWR0151")
 					(unit 1)
 				)
@@
 			)
 		)
-		(property "Footprint" "Package_TO_SOT_THT:TO-220-3_Vertical"
+		(property "Footprint" "Package_TO_SOT_SMD:TO-252-3_TabPin2"
 			(at 99.06 35.56 0)
 			(hide yes)
@@
 		(in_pos_files yes)
 		(dnp no)
-		(property "Reference" "#PWR0146"
+		(property "Reference" "#PWR0145"
 			(at 49.53 46.99 0)
 			(hide yes)
@@
 			(project "MY_POWERFULL_PLC_PCB"
 				(path "/69a480d6-fa06-4fdd-8ed7-9beeb2ac027a/ea39046e-ca02-46d1-9fd4-b85a58c0b80f/4e719e6a-f498-4860-85c2-d3c910fb7d70"
-					(reference "#PWR0146")
+					(reference "#PWR0145")
 					(unit 1)
 				)
 				(path "/69a480d6-fa06-4fdd-8ed7-9beeb2ac027a/ea39046e-ca02-46d1-9fd4-b85a58c0b80f/5918cb53-767b-4406-8a2b-be52ced64ae0"
-					(reference "#PWR0166")
+					(reference "#PWR0165")
 					(unit 1)
 				)
 				(path "/69a480d6-fa06-4fdd-8ed7-9beeb2ac027a/ea39046e-ca02-46d1-9fd4-b85a58c0b80f/6ec847d1-af3b-47e2-b394-844cce0f53eb"
-					(reference "#PWR0161")
+					(reference "#PWR0160")
 					(unit 1)
 				)
 				(path "/69a480d6-fa06-4fdd-8ed7-9beeb2ac027a/ea39046e-ca02-46d1-9fd4-b85a58c0b80f/938b05e1-ee13-4e84-85e5-d171a1a5f239"
-					(reference "#PWR0181")
+					(reference "#PWR0180")
 					(unit 1)
 				)
 				(path "/69a480d6-fa06-4fdd-8ed7-9beeb2ac027a/ea39046e-ca02-46d1-9fd4-b85a58c0b80f/94887116-e992-4614-87b1-1893944a34af"
-					(reference "#PWR0176")
+					(reference "#PWR0175")
 					(unit 1)
 				)
 				(path "/69a480d6-fa06-4fdd-8ed7-9beeb2ac027a/ea39046e-ca02-46d1-9fd4-b85a58c0b80f/976e15ae-69f2-46a4-92b9-157eb83b98b3"
-					(reference "#PWR0171")
+					(reference "#PWR0170")
 					(unit 1)
 				)
 				(path "/69a480d6-fa06-4fdd-8ed7-9beeb2ac027a/ea39046e-ca02-46d1-9fd4-b85a58c0b80f/9dcca28d-a41c-4e95-8119-28bf2da75604"
-					(reference "#PWR0156")
+					(reference "#PWR0155")
 					(unit 1)
 				)
 				(path "/69a480d6-fa06-4fdd-8ed7-9beeb2ac027a/ea39046e-ca02-46d1-9fd4-b85a58c0b80f/bdb5a479-48da-432b-97a9-55765e4484ff"
-					(reference "#PWR0151")
-					(unit 1)
-				)
+					(reference "#PWR0150")
+					(unit 1)
+				)
