File: .history/MCU_STM32.kicad_sch (KiCad schematic)
At the start: 4 parts, among them J10 Conn_02x20_Counter_Clockwise, J9 Conn_01x05

Commit message: 112
Parts:
- added J10, J11: Conn_02x07_Counter_Clockwise, Connector_PinSocket_2.54mm:PinSocket_2x07_P2.54mm_Horizontal, symbol Connector_Generic:Conn_02x07_Counter_Clockwise
- renumbered J10 to J12
Other:
- moved on the sheet: J12, J9, MOD1, U6

Commit message: 112
Parts:
- removed J10, J11: Conn_02x07_Counter_Clockwise, Connector_PinSocket_2.54mm:PinSocket_2x07_P2.54mm_Horizontal, symbol Connector_Generic:Conn_02x07_Counter_Clockwise
- removed J12: Conn_02x20_Counter_Clockwise, Connector_IDC:IDC-Header_2x25_P2.54mm_Vertical, symbol Connector_Generic:Conn_02x25_Odd_Even
- removed J9: Conn_01x05, Connector_PinHeader_2.54mm:PinHeader_1x07_P2.54mm_Vertical, symbol Connector_Generic:Conn_01x07
- added J14: Conn_02x20_Counter_Clockwise, Connector_PinSocket_2.54mm:PinSocket_2x28_P2.54mm_Vertical, symbol Connector_Generic:Conn_02x28_Odd_Even
- added J15: Conn_02x07_Counter_Clockwise, Connector_PinSocket_2.54mm:PinSocket_2x07_P2.54mm_Vertical, symbol Connector_Generic:Conn_02x07_Odd_Even
Connections:
- net +5V: now also MOD1.2 (+5V), MOD1.86 (5V), J14.1 (Pin_1), J14.27 (Pin_27), J14.28 (Pin_28)
- net AD7606_BUSY: now also J14.51 (Pin_51)
- net AD7606_CONVST: now also J14.54 (Pin_54)
- net AD7606_CS: now also J14.50 (Pin_50)
- net AD7606_MISO: now also J14.49 (Pin_49)
- net AD7606_RST: now also J14.52 (Pin_52)
- net AD7606_SCK: now also J14.53 (Pin_53)
- net DI_IN9_LOGIC10: now also J14.17 (Pin_17)
- net DI_IN9_LOGIC11: now also J14.15 (Pin_15)
- net DI_IN9_LOGIC12: now also J14.13 (Pin_13)
- net DI_IN9_LOGIC13: now also J14.11 (Pin_11)
- net DI_IN9_LOGIC14: now also J14.9 (Pin_9)
- net DI_IN9_LOGIC9: now also J14.19 (Pin_19)
- net DI_SLOW_LOGIC1: now also J14.43 (Pin_43)
- net DI_SLOW_LOGIC2: now also J14.41 (Pin_41)
- net DI_SLOW_LOGIC3: now also J14.39 (Pin_39)
- net DI_SLOW_LOGIC4: now also J14.37 (Pin_37)
- net DI_SLOW_LOGIC5: now also J14.35 (Pin_35)
- net DI_SLOW_LOGIC6: now also J14.33 (Pin_33)
- net DI_SLOW_LOGIC7: now also J14.31 (Pin_31)
- net DI_SLOW_LOGIC8: now also J14.29 (Pin_29)
- net DO_PWM_CTRL1: now also J14.30 (Pin_30)
- net DO_PWM_CTRL2: now also J14.32 (Pin_32)
- net DO_PWM_CTRL3: now also J14.34 (Pin_34)
- net DO_PWM_CTRL4: now also J14.36 (Pin_36)
- net DO_PWM_CTRL5: now also J14.38 (Pin_38)
- net DO_PWM_CTRL6: now also J14.40 (Pin_40)
- net DO_PWM_CTRL7: now also J14.42 (Pin_42)
- net DO_PWM_CTRL8: now also J14.44 (Pin_44)
- net DO_SLOW_CTRL1: now also J14.6 (Pin_6)
- net DO_SLOW_CTRL2: now also J14.8 (Pin_8)
- net DO_SLOW_CTRL3: now also J14.10 (Pin_10)
- net DO_SLOW_CTRL4: now also J14.12 (Pin_12)
- net DO_SLOW_CTRL5: now also J14.14 (Pin_14)
- net DO_SLOW_CTRL6: now also J14.16 (Pin_16)
- net DO_SLOW_CTRL7: now also J14.18 (Pin_18)
- net DO_SLOW_CTRL8: now also J14.20 (Pin_20)
- net ETH_TXD1: now reaches MOD1.43 (B13)
- net ETH_TXD1: now also J15.2 (Pin_2)
- net ETH_TXD0: now reaches MOD1.44 (B12)
- net ETH_TXD0: now also J15.3 (Pin_3)
- net +3V3: now reaches MOD1.46 (+3V3)
- net +3V3: now also MOD1.85 (3V3), J14.2 (Pin_2), J14.47 (Pin_47), J14.48 (Pin_48), J15.13 (Pin_13), J15.14 (Pin_14)
- net ETH_MDC: now reaches MOD1.56 (C1)
- net ETH_MDC: now also J15.9 (Pin_9)
- net ETH_REF_CLK: now reaches MOD1.62 (A1)
- net ETH_REF_CLK: now also J15.8 (Pin_8)
- net ETH_MDIO: now reaches MOD1.63 (A2)
- net ETH_MDIO: now also J15.10 (Pin_10)
- net ETH_CRS_DV: now reaches MOD1.68 (A7)
- net ETH_CRS_DV: now also J15.7 (Pin_7)
- net ETH_RXD0: now reaches MOD1.69 (C4)
- net ETH_RXD0: now also J15.6 (Pin_6)
- net ETH_RXD1: now reaches MOD1.70 (C5)
- net ETH_RXD1: now also J15.5 (Pin_5)
- net ETH_TX_EN: now reaches MOD1.84 (B11)
- net ETH_TX_EN: now also J15.4 (Pin_4)
- net Logic_GND renamed LOGIC_GND
- net LOGIC_GND: now also J14.21 (Pin_21), J14.22 (Pin_22), J14.23 (Pin_23), J14.24 (Pin_24), J14.25 (Pin_25), J14.26 (Pin_26), J14.3 (Pin_3), J14.4 (Pin_4), J14.45 (Pin_45), J14.46 (Pin_46), J14.5 (Pin_5), J14.7 (Pin_7), J15.1 (Pin_1), J15.11 (Pin_11), J15.12 (Pin_12)
Other:
- note added: "PA1 ETH_REF_CLK PA2 ETH_MDIO PA7 ETH_CRS_DV PB11 ETH_TX_EN PB12 ETH_TXD0 PB13 ETH_TXD1 PC1 ETH_MDC PC4 ETH_RXD0 PC5 ETH_RXD1"

Commit message: 112
Parts:
- added J11, J12: Conn_02x07_Counter_Clockwise, Connector_PinSocket_2.54mm:PinSocket_2x07_P2.54mm_Vertical, symbol Connector_Generic:Conn_02x07_Odd_Even
- renumbered J14 to J13, J15 to J14
Connections:
- net +3V3 renamed +3V3_Core
- net +3V3_Core: now also J11.1 (Pin_1), J11.11 (Pin_11), J11.13 (Pin_13), J11.3 (Pin_3), J11.5 (Pin_5), J11.7 (Pin_7), J11.9 (Pin_9)
- net +5V renamed +5V_Core
- net +5V_Core: now also J12.1 (Pin_1), J12.11 (Pin_11), J12.13 (Pin_13), J12.3 (Pin_3), J12.5 (Pin_5), J12.7 (Pin_7), J12.9 (Pin_9)
- net LOGIC_GND renamed GND_Core
- net GND_Core: now also J11.10 (Pin_10), J11.12 (Pin_12), J11.14 (Pin_14), J11.2 (Pin_2), J11.4 (Pin_4), J11.6 (Pin_6), J11.8 (Pin_8), J12.10 (Pin_10), J12.12 (Pin_12), J12.14 (Pin_14), J12.2 (Pin_2), J12.4 (Pin_4), J12.6 (Pin_6), J12.8 (Pin_8)
