File: .history/MY_POWERFULL_PLC_PCB.kicad_sch (KiCad schematic)
At the start: 6 parts, among them J1 DI_IN_Connector, J2 DI_IN_Connector, J3 DI_IN_Connector, J4 DI_IN_Connector, J5 DI_IN_Connector, J6 DI_IN_Connector

Commit message: 112
Parts:
- removed J4: DI_IN_Connector, Connector_Phoenix_MC:PhoenixContact_MC_1,5_10-G-3.81_1x10_P3.81mm_Horizontal, symbol Connector_Generic:Conn_01x09
- added H1, H2, H3, H4, H5, H6, H7, H8: MountingHole, MountingHole:MountingHole_3.2mm_M3_Pad, symbol Mechanical:MountingHole
- added J13, J2: Conn_02x20_Counter_Clockwise, Connector_IDC:IDC-Header_2x20_P2.54mm_Vertical, symbol Connector_Generic:Conn_02x20_Odd_Even
- added J3, J4, J9: Conn_02x20_Counter_Clockwise, Connector_IDC:IDC-Header_2x08_P2.54mm_Vertical, symbol Connector_Generic:Conn_02x08_Odd_Even
- added J6, J7: Conn_02x20_Counter_Clockwise, Connector_IDC:IDC-Header_2x06_P2.54mm_Vertical, symbol Connector_Generic:Conn_02x06_Odd_Even
- added J8: DI_IN_Connector, Connector_Phoenix_MC:PhoenixContact_MC_1,5_9-G-3.5_1x09_P3.50mm_Horizontal, symbol Connector_Generic:Conn_01x09
- added MOD1: (no value), MyModules:WeAct_STM32H743VIT6, symbol MyModules:WeAct_STM32H743VIT6
- added U1: (no value), MyModules:DAC8568_Module_57x52mm, symbol MyModules:Module_DAC8568_8CH
- added U2: (no value), MyModules:AD7606_Module_40x30mm, symbol MyModules:Module_AD7606_8CH
- J1: renamed from J5; footprint Connector_Phoenix_MC:PhoenixContact_MC_1,5_10-G-3.81_1x10_P3.81mm_Horizontal -> Connector_Phoenix_MC:PhoenixContact_MC_1,5_12-G-3.5_1x12_P3.50mm_Horizontal; symbol Connector_Generic:Conn_01x10 -> Connector_Generic:Conn_01x12
- J10: renamed from J3; footprint Connector_Phoenix_MC:PhoenixContact_MC_1,5_10-G-3.81_1x10_P3.81mm_Horizontal -> Connector_Phoenix_MC:PhoenixContact_MC_1,5_12-G-3.5_1x12_P3.50mm_Horizontal; symbol Connector_Generic:Conn_01x09 -> Connector_Generic:Conn_01x12
- J11: renamed from J6; footprint Connector_Phoenix_MC:PhoenixContact_MC_1,5_10-G-3.81_1x10_P3.81mm_Horizontal -> Connector_Phoenix_MC:PhoenixContact_MC_1,5_12-G-3.5_1x12_P3.50mm_Horizontal; symbol Connector_Generic:Conn_01x09 -> Connector_Generic:Conn_01x12
- J12: renamed from J2; footprint Connector_Phoenix_MC:PhoenixContact_MC_1,5_10-G-3.81_1x10_P3.81mm_Horizontal -> Connector_Phoenix_MC:PhoenixContact_MC_1,5_12-G-3.5_1x12_P3.50mm_Horizontal; symbol Connector_Generic:Conn_01x10 -> Connector_Generic:Conn_01x12
- J5: renamed from J1; footprint Connector_Phoenix_MC:PhoenixContact_MC_1,5_10-G-3.81_1x10_P3.81mm_Horizontal -> Connector_Phoenix_MC:PhoenixContact_MC_1,5_12-G-3.5_1x12_P3.50mm_Horizontal; symbol Connector_Generic:Conn_01x10 -> Connector_Generic:Conn_01x12
Connections:
- net DI_Channel7/DI_FIELD_IN is gone; now on net Field_GND: J1.2 (Pin_2)
- net DO_Channel/DO_OUT is gone; now on net +24V: J5.2 (Pin_2)
- net +24V: now also J11.1 (Pin_1), J11.11 (Pin_11), J11.2 (Pin_2), J5.11 (Pin_11), J5.12 (Pin_12); no longer J5.10 (Pin_10)
- net DO_OUT9: now reaches J11.3 (Pin_3)
- net DO_OUT10: now reaches J11.4 (Pin_4)
- net DO_OUT11: now reaches J11.5 (Pin_5)
- net DO_OUT12: now reaches J11.6 (Pin_6)
- net DO_OUT13: now reaches J11.7 (Pin_7)
- net DO_OUT14: now reaches J11.8 (Pin_8)
- net DO_OUT15: now reaches J11.9 (Pin_9)
- net Field_GND: now reaches J12.1 (Pin_1)
- net Field_GND: now also J1.1 (Pin_1), J1.11 (Pin_11), J1.12 (Pin_12), J11.12 (Pin_12), J12.11 (Pin_11), J12.12 (Pin_12), J12.2 (Pin_2), J7.1 (Pin_1), J7.3 (Pin_3), J7.5 (Pin_5), J7.7 (Pin_7), J8.9 (Pin_9)
- net DI_IN16: now reaches J12.10 (Pin_10)
- net DI_IN9: now reaches J12.3 (Pin_3)
- net DI_IN10: now reaches J12.4 (Pin_4)
- net DI_IN11: now reaches J12.5 (Pin_5)
- net DI_IN12: now reaches J12.6 (Pin_6)
- net DI_IN13: now reaches J12.7 (Pin_7)
- net DI_IN14: now reaches J12.8 (Pin_8)
- net DI_IN15: now reaches J12.9 (Pin_9)
- net DI_Channel/DI_FIELD_IN renamed DI_IN7
- net DI_Channel1/DI_FIELD_IN renamed DI_IN6
- net DI_Channel2/DI_FIELD_IN renamed DI_IN5
- net DI_Channel3/DI_FIELD_IN renamed DI_IN4
- net DI_Channel4/DI_FIELD_IN renamed DI_IN3
- net DI_Channel5/DI_FIELD_IN renamed DI_IN2
- net DI_Channel6/DI_FIELD_IN renamed DI_IN1
- net DO_Channel1/DO_OUT renamed DO_OUT1
- net DO_Channel2/DO_OUT renamed DO_OUT2
- net DO_Channel3/DO_OUT renamed DO_OUT3
- net DO_Channel4/DO_OUT renamed DO_OUT4
- net DO_Channel5/DO_OUT renamed DO_OUT5
- net DO_Channel6/DO_OUT renamed DO_OUT6
- net DO_Channel7/DO_OUT renamed DO_OUT7
- net FIELD_GND renamed DI_IN8
- net DI_IN8: no longer J1.1 (Pin_1)
- new net: J13.1 (Pin_1), MOD1.1 (GND)
- new net: J13.3 (Pin_3), MOD1.2 (+5V)
- new net: J6.1 (Pin_1), J6.3 (Pin_3), J6.5 (Pin_5), J6.7 (Pin_7), U1.17 (GND), U1.8 (GND)
- new net: J6.10 (Pin_10), U1.12 (VD)
- new net: J6.11 (Pin_11), U1.10 (VB)
- new net: J6.12 (Pin_12), U1.11 (VC)
- new net: J6.2 (Pin_2), U1.16 (VH)
- new net: J6.4 (Pin_4), U1.15 (VG)
- new net: J6.6 (Pin_6), U1.14 (VF)
- new net: J6.8 (Pin_8), U1.13 (VE)
- new net: J6.9 (Pin_9), U1.9 (VA)
- new net: J7.10 (Pin_10), J8.4 (Pin_4)
- new net: J7.11 (Pin_11), J8.2 (Pin_2)
- new net: J7.12 (Pin_12), J8.3 (Pin_3)
- new net: J7.2 (Pin_2), J8.8 (Pin_8)
- new net: J7.4 (Pin_4), J8.7 (Pin_7)
- new net: J7.6 (Pin_6), J8.6 (Pin_6)
- new net: J7.8 (Pin_8), J8.5 (Pin_5)
- new net: J7.9 (Pin_9), J8.1 (Pin_1)
- new net DI_IN9_LOGIC10: J2.14 (Pin_14)
- new net DI_IN9_LOGIC11: J2.12 (Pin_12)
- new net DI_IN9_LOGIC12: J2.10 (Pin_10)
- new net DI_IN9_LOGIC13: J2.8 (Pin_8)
- new net DI_IN9_LOGIC14: J2.6 (Pin_6)
- new net DI_IN9_LOGIC15: J2.4 (Pin_4)
- new net DI_IN9_LOGIC16: J2.2 (Pin_2)
- new net DI_IN9_LOGIC9: J2.16 (Pin_16)
- new net DI_SLOW_LOGIC1: J2.32 (Pin_32)
- new net DI_SLOW_LOGIC2: J2.30 (Pin_30)
- new net DI_SLOW_LOGIC3: J2.28 (Pin_28)
- new net DI_SLOW_LOGIC4: J2.26 (Pin_26)
- new net DI_SLOW_LOGIC5: J2.24 (Pin_24)
- new net DI_SLOW_LOGIC6: J2.22 (Pin_22)
- new net DI_SLOW_LOGIC7: J2.20 (Pin_20)
- new net DI_SLOW_LOGIC8: J2.18 (Pin_18)
- new net DO_OUT16: J11.10 (Pin_10)
- new net DO_OUT8: J5.10 (Pin_10)
- new net DO_PWM_CTRL1: J2.17 (Pin_17)
- new net DO_PWM_CTRL2: J2.19 (Pin_19)
- new net DO_PWM_CTRL3: J2.21 (Pin_21)
- new net DO_PWM_CTRL4: J2.23 (Pin_23)
- new net DO_PWM_CTRL5: J2.25 (Pin_25)
- new net DO_PWM_CTRL6: J2.27 (Pin_27)
- new net DO_PWM_CTRL7: J2.29 (Pin_29)
- new net DO_PWM_CTRL8: J2.31 (Pin_31)
- new net DO_SLOW_CTRL1: J2.1 (Pin_1)
- new net DO_SLOW_CTRL2: J2.3 (Pin_3)
- new net DO_SLOW_CTRL3: J2.5 (Pin_5)
- new net DO_SLOW_CTRL4: J2.7 (Pin_7)
- new net DO_SLOW_CTRL5: J2.9 (Pin_9)
- new net DO_SLOW_CTRL6: J2.11 (Pin_11)
- new net DO_SLOW_CTRL7: J2.13 (Pin_13)
- new net DO_SLOW_CTRL8: J2.15 (Pin_15)
Other:
- sheet 02_POWER_24V_5V renamed 02_POWER_5V
- sheet 03_POWER_5V_3V3 renamed 03_POWER_3V3
- removed sheet DI_Channel
- removed sheet DI_Channel1
- removed sheet DI_Channel2
- removed sheet DI_Channel3
- removed sheet DI_Channel4
- removed sheet DI_Channel5
- removed sheet DI_Channel6
- removed sheet DI_Channel7
- removed sheet DO_Channel
- removed sheet DO_Channel1
- removed sheet DO_Channel2
- removed sheet DO_Channel3
- removed sheet DO_Channel4
- removed sheet DO_Channel5
- removed sheet DO_Channel6
- removed sheet DO_Channel7
- added sheet DI_FAST_GROUP (DI_FAST_GROUP.kicad_sch)
- added sheet DI_SLOW_GROUP (DI_SLOW_GROUP.kicad_sch)
- added sheet DO_FAST_PWM (DO_FAST_PWM.kicad_sch)
- added sheet DO_GROUP (DO_GROUP.kicad_sch)

Commit message: 112
Parts:
- removed J10: DI_IN_Connector, Connector_Phoenix_MC:PhoenixContact_MC_1,5_12-G-3.5_1x12_P3.50mm_Horizontal, symbol Connector_Generic:Conn_01x12
- removed J13, J2: Conn_02x20_Counter_Clockwise, Connector_IDC:IDC-Header_2x20_P2.54mm_Vertical, symbol Connector_Generic:Conn_02x20_Odd_Even
- removed J3, J4, J9: Conn_02x20_Counter_Clockwise, Connector_IDC:IDC-Header_2x08_P2.54mm_Vertical, symbol Connector_Generic:Conn_02x08_Odd_Even
- removed J6, J7: Conn_02x20_Counter_Clockwise, Connector_IDC:IDC-Header_2x06_P2.54mm_Vertical, symbol Connector_Generic:Conn_02x06_Odd_Even
- removed MOD1: (no value), MyModules:WeAct_STM32H743VIT6, symbol MyModules:WeAct_STM32H743VIT6
- removed U1: (no value), MyModules:DAC8568_Module_57x52mm, symbol MyModules:Module_DAC8568_8CH
- removed U2: (no value), MyModules:AD7606_Module_40x30mm, symbol MyModules:Module_AD7606_8CH
- added J2: Conn_02x20_Counter_Clockwise, Connector_IDC:IDC-Header_2x25_P2.54mm_Vertical, symbol Connector_Generic:Conn_02x25_Odd_Even
- added J4: Conn_02x08_Counter_Clockwise, Connector_PinSocket_2.54mm:PinSocket_2x08_P2.54mm_Vertical_SMD, symbol Connector_Generic:Conn_02x08_Counter_Clockwise
- added J7: DI_IN_Connector, Connector_Phoenix_MC:PhoenixContact_MC_1,5_12-G-3.5_1x12_P3.50mm_Horizontal, symbol Connector_Generic:Conn_01x12
- added U1: (no value), MyModules:AD7606_Module_40x30mm, symbol MyModules:Module_AD7606_8CH
- J8: footprint Connector_Phoenix_MC:PhoenixContact_MC_1,5_9-G-3.5_1x09_P3.50mm_Horizontal -> Connector_Phoenix_MC:PhoenixContact_MC_1,5_12-G-3.5_1x12_P3.50mm_Horizontal; symbol Connector_Generic:Conn_01x09 -> Connector_Generic:Conn_01x12
- renumbered J5 to J3, J11 to J5, J12 to J6
Connections:
- net DI_IN15 is gone; now on net DI_IN12: J6.9 (Pin_9)
- net DI_IN16 is gone; now on net DI_IN13: J6.10 (Pin_10)
- net DI_IN1: now also J1.10 (Pin_10); no longer J1.3 (Pin_3)
- net DI_IN10: now also J6.7 (Pin_7); no longer J6.4 (Pin_4)
- net DI_IN11: now also J6.8 (Pin_8); no longer J6.5 (Pin_5)
- net DI_IN12: no longer J6.6 (Pin_6)
- net DI_IN13: no longer J6.7 (Pin_7)
- net DI_IN14: now also J6.11 (Pin_11); no longer J6.8 (Pin_8)
- net DI_IN2: now also J1.11 (Pin_11); no longer J1.4 (Pin_4)
- net DI_IN3: now also J1.12 (Pin_12); no longer J1.5 (Pin_5)
- net DI_IN4: now also J6.1 (Pin_1); no longer J1.6 (Pin_6)
- net DI_IN5: now also J6.2 (Pin_2); no longer J1.7 (Pin_7)
- net DI_IN6: now also J6.3 (Pin_3); no longer J1.8 (Pin_8)
- net DI_IN7: now also J6.4 (Pin_4); no longer J1.9 (Pin_9)
- net DI_IN8: now also J6.5 (Pin_5); no longer J1.10 (Pin_10)
- net DI_IN9: now also J6.6 (Pin_6); no longer J6.3 (Pin_3)
- net DI_IN9_LOGIC10: now also J2.14 (Pin_14)
- net DI_IN9_LOGIC11: now also J2.12 (Pin_12)
- net DI_IN9_LOGIC12: now also J2.10 (Pin_10)
- net DI_IN9_LOGIC13: now also J2.8 (Pin_8)
- net DI_IN9_LOGIC14: now also J2.6 (Pin_6)
- net DI_IN9_LOGIC9: now also J2.16 (Pin_16)
- net DI_SLOW_LOGIC1: now also J2.40 (Pin_40)
- net DI_SLOW_LOGIC2: now also J2.38 (Pin_38)
- net DI_SLOW_LOGIC3: now also J2.36 (Pin_36)
- net DI_SLOW_LOGIC4: now also J2.34 (Pin_34)
- net DI_SLOW_LOGIC5: now also J2.32 (Pin_32)
- net DI_SLOW_LOGIC6: now also J2.30 (Pin_30)
- net DI_SLOW_LOGIC7: now also J2.28 (Pin_28)
- net DI_SLOW_LOGIC8: now also J2.26 (Pin_26)
- net DO_PWM_CTRL1: now also J2.25 (Pin_25)
- net DO_PWM_CTRL2: now also J2.27 (Pin_27)
- net DO_PWM_CTRL3: now also J2.29 (Pin_29)
- net DO_PWM_CTRL4: now also J2.31 (Pin_31)
- net DO_PWM_CTRL5: now also J2.33 (Pin_33)
- net DO_PWM_CTRL6: now also J2.35 (Pin_35)
- net DO_PWM_CTRL7: now also J2.37 (Pin_37)
- net DO_PWM_CTRL8: now also J2.39 (Pin_39)
- net DO_SLOW_CTRL1: now also J2.1 (Pin_1)
- net DO_SLOW_CTRL2: now also J2.3 (Pin_3)
- net DO_SLOW_CTRL3: now also J2.5 (Pin_5)
- net DO_SLOW_CTRL4: now also J2.7 (Pin_7)
- net DO_SLOW_CTRL5: now also J2.9 (Pin_9)
- net DO_SLOW_CTRL6: now also J2.11 (Pin_11)
- net DO_SLOW_CTRL7: now also J2.13 (Pin_13)
- net DO_SLOW_CTRL8: now also J2.15 (Pin_15)
- net Field_GND: no longer J1.1 (Pin_1), J1.11 (Pin_11), J1.12 (Pin_12), J1.2 (Pin_2), J6.1 (Pin_1), J6.11 (Pin_11), J6.2 (Pin_2), J8.9 (Pin_9)
- new net +3V3: U1.14 (VIO)
- new net +5V: U1.2 (+5V), U1.6 (RANGE)
- new net AD7606_BUSY: J2.48 (Pin_48), U1.11 (BUSY)
- new net AD7606_CONVST: J2.49 (Pin_49), U1.7 (CVA), U1.8 (CVB)
- new net AD7606_CS: J2.45 (Pin_45), U1.12 (CS)
- new net AD7606_MISO: J2.46 (Pin_46), U1.21 (DB7_MISO)
- new net AD7606_RST: J2.47 (Pin_47), U1.10 (RST)
- new net AD7606_SCK: J2.50 (Pin_50), U1.9 (RD_SCLK)
- new net AD7606_V1: J1.9 (Pin_9), U1.31 (V1)
- new net AD7606_V2: J1.8 (Pin_8), U1.33 (V2)
- new net AD7606_V3: J1.7 (Pin_7), U1.35 (V3)
- new net AD7606_V4: J1.6 (Pin_6), U1.37 (V4)
- new net AD7606_V5: J1.5 (Pin_5), U1.39 (V5)
- new net AD7606_V6: J1.4 (Pin_4), U1.41 (V6)
- new net AD7606_V7: J1.3 (Pin_3), U1.43 (V7)
- new net AD7606_V8: J1.2 (Pin_2), U1.45 (V8)
- new net Logic_GND: J2.17 (Pin_17), J2.18 (Pin_18), J2.19 (Pin_19), J2.2 (Pin_2), J2.20 (Pin_20), J2.21 (Pin_21), J2.22 (Pin_22), J2.23 (Pin_23), J2.24 (Pin_24), J2.4 (Pin_4), U1.1 (GND), U1.3 (OS0), U1.32 (GND), U1.34 (GND), U1.36 (GND), U1.38 (GND), U1.4 (OS1), U1.40 (GND), U1.42 (GND), U1.44 (GND), U1.46 (GND), U1.5 (OS2)
Other:
- added sheet MCU_STM32 (MCU_STM32.kicad_sch)
- sheet DI_FAST_GROUP ports: added none; removed DI_FAST_IN7, DI_FAST_IN8, DI_FAST_LOGIC7, DI_FAST_LOGIC8
- moved on the sheet: J5, J6

Commit message: 112
Parts:
- removed H1, H2, H3, H4, H5, H6, H7, H8: MountingHole, MountingHole:MountingHole_3.2mm_M3_Pad, symbol Mechanical:MountingHole
Connections:
- net +24V: no longer J3.11 (Pin_11), J3.12 (Pin_12), J5.11 (Pin_11)
- net DO_OUT10: now also J5.5 (Pin_5); no longer J5.4 (Pin_4)
- net DO_OUT11: now also J5.4 (Pin_4); no longer J5.5 (Pin_5)
- net DO_OUT12: now also J5.7 (Pin_7); no longer J5.6 (Pin_6)
- net DO_OUT13: now also J5.6 (Pin_6); no longer J5.7 (Pin_7)
- net DO_OUT14: now also J5.9 (Pin_9); no longer J5.8 (Pin_8)
- net DO_OUT15: now also J5.8 (Pin_8); no longer J5.9 (Pin_9)
- net Field_GND: now also J3.11 (Pin_11), J3.12 (Pin_12), J5.11 (Pin_11)
- net Logic_GND: now also J2.41 (Pin_41), J2.42 (Pin_42), J2.43 (Pin_43), J2.44 (Pin_44)
Other:
- moved on the sheet: J2

Commit message: 112
Parts:
- removed J2: Conn_02x20_Counter_Clockwise, Connector_IDC:IDC-Header_2x25_P2.54mm_Vertical, symbol Connector_Generic:Conn_02x25_Odd_Even
- removed J4: Conn_02x08_Counter_Clockwise, Connector_PinSocket_2.54mm:PinSocket_2x08_P2.54mm_Vertical_SMD, symbol Connector_Generic:Conn_02x08_Counter_Clockwise
- removed J8: DI_IN_Connector, Connector_Phoenix_MC:PhoenixContact_MC_1,5_12-G-3.5_1x12_P3.50mm_Horizontal, symbol Connector_Generic:Conn_01x12
- added J1: DI_IN_Connector, Connector_Phoenix_MC:PhoenixContact_MC_1,5_2-G-3.5_1x02_P3.50mm_Horizontal, symbol Connector_Generic:Conn_01x02
- added J10, J8, J9: Conn_02x07_Counter_Clockwise, Connector_PinHeader_2.54mm:PinHeader_2x07_P2.54mm_Vertical, symbol Connector_Generic:Conn_02x07_Odd_Even
- added J3: Conn_02x20_Counter_Clockwise, Connector_PinHeader_2.54mm:PinHeader_2x28_P2.54mm_Vertical, symbol Connector_Generic:Conn_02x28_Odd_Even
- added J5: Conn_02x07_Counter_Clockwise, Connector_PinSocket_2.54mm:PinSocket_2x07_P2.54mm_Horizontal, symbol Connector_Generic:Conn_02x07_Odd_Even
- added J6, J7: Conn_02x07_Counter_Clockwise, Connector_PinSocket_2.54mm:PinSocket_2x07_P2.54mm_Vertical, symbol Connector_Generic:Conn_02x07_Odd_Even
- J11: renamed from J5; footprint Connector_Phoenix_MC:PhoenixContact_MC_1,5_12-G-3.5_1x12_P3.50mm_Horizontal -> Connector_Phoenix_MC:PhoenixContact_MC_1,5_8-G-3.5_1x08_P3.50mm_Horizontal; symbol Connector_Generic:Conn_01x12 -> Connector_Generic:Conn_01x08
- J12: renamed from J6; footprint Connector_Phoenix_MC:PhoenixContact_MC_1,5_12-G-3.5_1x12_P3.50mm_Horizontal -> Connector_Phoenix_MC:PhoenixContact_MC_1,5_16-G-3.5_1x16_P3.50mm_Horizontal; symbol Connector_Generic:Conn_01x12 -> Connector_Generic:Conn_01x16
- J2: renamed from J1; footprint Connector_Phoenix_MC:PhoenixContact_MC_1,5_12-G-3.5_1x12_P3.50mm_Horizontal -> Connector_Phoenix_MC:PhoenixContact_MC_1,5_16-G-3.5_1x16_P3.50mm_Horizontal; symbol Connector_Generic:Conn_01x12 -> Connector_Generic:Conn_01x16
- J4: renamed from J3; footprint Connector_Phoenix_MC:PhoenixContact_MC_1,5_12-G-3.5_1x12_P3.50mm_Horizontal -> Connector_Phoenix_MC:PhoenixContact_MC_1,5_16-G-3.5_1x16_P3.50mm_Horizontal; symbol Connector_Generic:Conn_01x12 -> Connector_Generic:Conn_01x16
- renumbered J7 to J13
Connections:
- net +24V: now also J11.6 (Pin_6), J11.7 (Pin_7), J11.8 (Pin_8), J12.16 (Pin_16), J2.16 (Pin_16), J2.4 (Pin_4), J2.5 (Pin_5), J2.6 (Pin_6), J1.2 (Pin_2); no longer J11.1 (Pin_1), J11.2 (Pin_2), J4.2 (Pin_2)
- net +3V3: now also J10.13 (Pin_13), J10.14 (Pin_14), J3.47 (Pin_47), J3.48 (Pin_48), J5.13 (Pin_13), J5.14 (Pin_14), J6.1 (Pin_1), J6.11 (Pin_11), J6.13 (Pin_13), J6.3 (Pin_3), J6.5 (Pin_5), J6.7 (Pin_7), J6.9 (Pin_9), J8.1 (Pin_1), J8.11 (Pin_11), J8.13 (Pin_13), J8.3 (Pin_3), J8.5 (Pin_5), J8.7 (Pin_7), J8.9 (Pin_9)
- net +5V: now also J3.27 (Pin_27), J3.28 (Pin_28), J7.1 (Pin_1), J7.11 (Pin_11), J7.13 (Pin_13), J7.3 (Pin_3), J7.5 (Pin_5), J7.7 (Pin_7), J7.9 (Pin_9), J9.1 (Pin_1), J9.11 (Pin_11), J9.13 (Pin_13), J9.3 (Pin_3), J9.5 (Pin_5), J9.7 (Pin_7), J9.9 (Pin_9)
- net AD7606_BUSY: now also J3.52 (Pin_52)
- net AD7606_CONVST: now also J3.53 (Pin_53)
- net AD7606_CS: now also J3.49 (Pin_49)
- net AD7606_MISO: now also J3.50 (Pin_50)
- net AD7606_RST: now also J3.51 (Pin_51)
- net AD7606_SCK: now also J3.54 (Pin_54)
- net AD7606_V1: now also J2.14 (Pin_14); no longer J2.9 (Pin_9)
- net AD7606_V2: now also J2.13 (Pin_13); no longer J2.8 (Pin_8)
- net AD7606_V3: now also J2.12 (Pin_12); no longer J2.7 (Pin_7)
- net AD7606_V4: now also J2.11 (Pin_11); no longer J2.6 (Pin_6)
- net AD7606_V5: now also J2.10 (Pin_10); no longer J2.5 (Pin_5)
- net AD7606_V6: now also J2.9 (Pin_9); no longer J2.4 (Pin_4)
- net AD7606_V7: now also J2.8 (Pin_8); no longer J2.3 (Pin_3)
- net AD7606_V8: now also J2.7 (Pin_7); no longer J2.2 (Pin_2)
- net DI_IN1: now also J12.1 (Pin_1); no longer J2.10 (Pin_10)
- net DI_IN10: now also J12.10 (Pin_10); no longer J12.7 (Pin_7)
- net DI_IN11: now also J12.11 (Pin_11); no longer J12.8 (Pin_8)
- net DI_IN12: now also J12.12 (Pin_12); no longer J12.9 (Pin_9)
- net DI_IN13: now also J12.13 (Pin_13); no longer J12.10 (Pin_10)
- net DI_IN14: now also J12.14 (Pin_14); no longer J12.11 (Pin_11)
- net DI_IN2: now also J12.2 (Pin_2); no longer J2.11 (Pin_11)
- net DI_IN3: now also J12.3 (Pin_3); no longer J2.12 (Pin_12)
- net DI_IN4: now also J12.4 (Pin_4); no longer J12.1 (Pin_1)
- net DI_IN5: now also J12.5 (Pin_5); no longer J12.2 (Pin_2)
- net DI_IN6: now also J12.6 (Pin_6); no longer J12.3 (Pin_3)
- net DI_IN7: now also J12.7 (Pin_7); no longer J12.4 (Pin_4)
- net DI_IN8: now also J12.8 (Pin_8); no longer J12.5 (Pin_5)
- net DI_IN9: now also J12.9 (Pin_9); no longer J12.6 (Pin_6)
- net DI_IN9_LOGIC10: now also J3.18 (Pin_18)
- net DI_IN9_LOGIC11: now also J3.16 (Pin_16)
- net DI_IN9_LOGIC12: now also J3.14 (Pin_14)
- net DI_IN9_LOGIC13: now also J3.12 (Pin_12)
- net DI_IN9_LOGIC14: now also J3.10 (Pin_10)
- net DI_IN9_LOGIC9: now also J3.20 (Pin_20)
- net DI_SLOW_LOGIC1: now also J3.44 (Pin_44)
- net DI_SLOW_LOGIC2: now also J3.42 (Pin_42)
- net DI_SLOW_LOGIC3: now also J3.40 (Pin_40)
- net DI_SLOW_LOGIC4: now also J3.38 (Pin_38)
- net DI_SLOW_LOGIC5: now also J3.36 (Pin_36)
- net DI_SLOW_LOGIC6: now also J3.34 (Pin_34)
- net DI_SLOW_LOGIC7: now also J3.32 (Pin_32)
- net DI_SLOW_LOGIC8: now also J3.30 (Pin_30)
- net DO_OUT10: now also J4.13 (Pin_13); no longer J11.5 (Pin_5)
- net DO_OUT11: now also J4.12 (Pin_12); no longer J11.4 (Pin_4)
- net DO_OUT12: now also J4.15 (Pin_15); no longer J11.7 (Pin_7)
- net DO_OUT13: now also J4.14 (Pin_14); no longer J11.6 (Pin_6)
- net DO_OUT14: now also J11.1 (Pin_1); no longer J11.9 (Pin_9)
- net DO_OUT15: now also J4.16 (Pin_16); no longer J11.8 (Pin_8)
- net DO_OUT16: now also J11.2 (Pin_2); no longer J11.10 (Pin_10)
- net DO_OUT9: now also J4.11 (Pin_11); no longer J11.3 (Pin_3)
- net DO_PWM_CTRL1: now also J3.29 (Pin_29)
- net DO_PWM_CTRL2: now also J3.31 (Pin_31)
- net DO_PWM_CTRL3: now also J3.33 (Pin_33)
- net DO_PWM_CTRL4: now also J3.35 (Pin_35)
- net DO_PWM_CTRL5: now also J3.37 (Pin_37)
- net DO_PWM_CTRL6: now also J3.39 (Pin_39)
- net DO_PWM_CTRL7: now also J3.41 (Pin_41)
- net DO_PWM_CTRL8: now also J3.43 (Pin_43)
- net DO_SLOW_CTRL1: now also J3.5 (Pin_5)
- net DO_SLOW_CTRL2: now also J3.7 (Pin_7)
- net DO_SLOW_CTRL3: now also J3.9 (Pin_9)
- net DO_SLOW_CTRL4: now also J3.11 (Pin_11)
- net DO_SLOW_CTRL5: now also J3.13 (Pin_13)
- net DO_SLOW_CTRL6: now also J3.15 (Pin_15)
- net DO_SLOW_CTRL7: now also J3.17 (Pin_17)
- net DO_SLOW_CTRL8: now also J3.19 (Pin_19)
- net Field_GND: now also J11.3 (Pin_3), J11.4 (Pin_4), J11.5 (Pin_5), J12.15 (Pin_15), J2.1 (Pin_1), J2.15 (Pin_15), J2.2 (Pin_2), J2.3 (Pin_3), J4.2 (Pin_2), J1.1 (Pin_1); no longer J11.11 (Pin_11), J11.12 (Pin_12), J12.12 (Pin_12), J4.11 (Pin_11), J4.12 (Pin_12)
- net Logic_GND: now also J10.1 (Pin_1), J10.11 (Pin_11), J10.12 (Pin_12), J3.21 (Pin_21), J3.22 (Pin_22), J3.23 (Pin_23), J3.24 (Pin_24), J3.25 (Pin_25), J3.26 (Pin_26), J3.45 (Pin_45), J3.46 (Pin_46), J3.6 (Pin_6), J3.8 (Pin_8), J5.1 (Pin_1), J5.11 (Pin_11), J5.12 (Pin_12), J6.10 (Pin_10), J6.12 (Pin_12), J6.14 (Pin_14), J6.2 (Pin_2), J6.4 (Pin_4), J6.6 (Pin_6), J6.8 (Pin_8), J7.10 (Pin_10), J7.12 (Pin_12), J7.14 (Pin_14), J7.2 (Pin_2), J7.4 (Pin_4), J7.6 (Pin_6), J7.8 (Pin_8), J8.10 (Pin_10), J8.12 (Pin_12), J8.14 (Pin_14), J8.2 (Pin_2), J8.4 (Pin_4), J8.6 (Pin_6), J8.8 (Pin_8), J9.10 (Pin_10), J9.12 (Pin_12), J9.14 (Pin_14), J9.2 (Pin_2), J9.4 (Pin_4), J9.6 (Pin_6), J9.8 (Pin_8); no longer U1.32 (GND), U1.34 (GND), U1.36 (GND), U1.38 (GND), U1.40 (GND), U1.42 (GND), U1.44 (GND), U1.46 (GND)
- new net ETH_CRS_DV: J10.7 (Pin_7), J5.7 (Pin_7)
- new net ETH_MDC: J10.9 (Pin_9), J5.9 (Pin_9)
- new net ETH_MDIO: J10.10 (Pin_10), J5.10 (Pin_10)
- new net ETH_REF_CLK: J10.8 (Pin_8), J5.8 (Pin_8)
- new net ETH_RXD0: J10.6 (Pin_6), J5.6 (Pin_6)
- new net ETH_RXD1: J10.5 (Pin_5), J5.5 (Pin_5)
- new net ETH_TXD0: J10.3 (Pin_3), J5.3 (Pin_3)
- new net ETH_TXD1: J10.2 (Pin_2), J5.2 (Pin_2)
- new net ETH_TX_EN: J10.4 (Pin_4), J5.4 (Pin_4)
- new net FIELD_GND: U1.32 (GND), U1.34 (GND), U1.36 (GND), U1.38 (GND), U1.40 (GND), U1.42 (GND), U1.44 (GND), U1.46 (GND)

Commit message: 112
Parts:
- removed J13: DI_IN_Connector, Connector_Phoenix_MC:PhoenixContact_MC_1,5_12-G-3.5_1x12_P3.50mm_Horizontal, symbol Connector_Generic:Conn_01x12
- removed J6, J7: Conn_02x07_Counter_Clockwise, Connector_PinSocket_2.54mm:PinSocket_2x07_P2.54mm_Vertical, symbol Connector_Generic:Conn_02x07_Odd_Even
- renumbered J12 to J10, J11 to J5, J5 to J6, J8 to J7, J9 to J8, J10 to J9
Connections:
- net Logic_GND is gone; now on net FIELD_GND: J3.21 (Pin_21), J3.22 (Pin_22), J3.23 (Pin_23), J3.24 (Pin_24), J3.25 (Pin_25), J3.26 (Pin_26), J3.45 (Pin_45), J3.46 (Pin_46), J3.6 (Pin_6), J3.8 (Pin_8), J6.1 (Pin_1), J6.11 (Pin_11), J6.12 (Pin_12), J7.10 (Pin_10), J7.12 (Pin_12), J7.14 (Pin_14), J7.2 (Pin_2), J7.4 (Pin_4), J7.6 (Pin_6), J7.8 (Pin_8), J8.10 (Pin_10), J8.12 (Pin_12), J8.14 (Pin_14), J8.2 (Pin_2), J8.4 (Pin_4), J8.6 (Pin_6), J8.8 (Pin_8), J9.1 (Pin_1), J9.11 (Pin_11), J9.12 (Pin_12), U1.1 (GND), U1.3 (OS0), U1.4 (OS1), U1.5 (OS2)
- net +24V: no longer J5.6 (Pin_6), J5.7 (Pin_7), J5.8 (Pin_8)
- net +3V3: now also J3.4 (Pin_4)
- net +5V: now also J3.2 (Pin_2), J3.55 (Pin_55); no longer J8.11 (Pin_11), J8.13 (Pin_13)
- net DO_OUT10: now also J4.16 (Pin_16); no longer J4.13 (Pin_13)
- net DO_OUT12: now also J5.4 (Pin_4); no longer J4.15 (Pin_15)
- net DO_OUT13: now also J4.15 (Pin_15); no longer J4.14 (Pin_14)
- net DO_OUT14: now also J5.7 (Pin_7); no longer J5.1 (Pin_1)
- net DO_OUT15: now also J5.3 (Pin_3); no longer J4.16 (Pin_16)
- net DO_OUT16: now also J5.8 (Pin_8); no longer J5.2 (Pin_2)
- net DO_PWM_CTRL2: now also J3.33 (Pin_33); no longer J3.31 (Pin_31)
- net DO_PWM_CTRL3: now also J3.31 (Pin_31); no longer J3.33 (Pin_33)
- net DO_PWM_CTRL4: now also J3.37 (Pin_37); no longer J3.35 (Pin_35)
- net DO_PWM_CTRL5: now also J3.35 (Pin_35); no longer J3.37 (Pin_37)
- net DO_PWM_CTRL6: now also J3.41 (Pin_41); no longer J3.39 (Pin_39)
- net DO_PWM_CTRL7: now also J3.39 (Pin_39); no longer J3.41 (Pin_41)
- net FIELD_GND: now also J3.1 (Pin_1), J3.3 (Pin_3), J3.56 (Pin_56), J8.11 (Pin_11), J8.13 (Pin_13)
- net Field_GND: no longer J5.3 (Pin_3), J5.4 (Pin_4), J5.5 (Pin_5)
Other:
- moved on the sheet: J5
