File: .history/MY_POWERFULL_PLC_PCB.kicad_pcb (KiCad board)
At the start: 2 copper layers, 230 x 90 mm, 115 parts, among them J1 DI_IN_Connector, J2 DI_IN_Connector, J3 DI_IN_Connector, J4 DI_IN_Connector, J5 DI_IN_Connector, J6 DI_IN_Connector, J7 Conn_01x02, Q1 NMOS, Q2 NMOS, Q3 NMOS, Q4 NMOS, Q5 NMOS, Q6 NMOS, Q7 NMOS, Q8 NMOS, Q9 Q_PMOS, U1 LTV-357T, U10 LTV-357T, U11 LTV-357T, U12 LTV-357T, U13 LTV-357T, U14 LTV-357T, U15 LTV-357T, U16 LTV-357T, U17 LMR51430, U18 AP7361C-33E, U2 LTV-357T, U3 LTV-357T, U4 LTV-357T, U5 LTV-357T, U6 LTV-357T, U7 LTV-357T, U8 LTV-357T, U9 LTV-357T

Commit message: 112
Parts:
- added C10: 100nF, Capacitor_SMD:C_0805_2012Metric, B.Cu at (63.7, 132.1)
- added C11: 100nF, Capacitor_SMD:C_0805_2012Metric, B.Cu at (62.7, 134.8)
- added C12: 1uF, Capacitor_SMD:C_0805_2012Metric, B.Cu at (61.7, 132.1)
- added C13: 100nF, Capacitor_SMD:C_0805_2012Metric, B.Cu at (57.7, 132.1)
- added C14: 100nF, Capacitor_SMD:C_0805_2012Metric, B.Cu at (56.6, 134.8)
- added C15: 1uF, Capacitor_SMD:C_0805_2012Metric, B.Cu at (55.7, 132.1)
- added C16: 100nF, Capacitor_SMD:C_0805_2012Metric, B.Cu at (51.7, 132.1)
- added C17: 100nF, Capacitor_SMD:C_0805_2012Metric, B.Cu at (50.6, 134.8)
- added C18: 1uF, Capacitor_SMD:C_0805_2012Metric, B.Cu at (49.7, 132.1)
- added C19: 100nF, Capacitor_SMD:C_0805_2012Metric, B.Cu at (120.9, 130.3)
- added C20: 100nF, Capacitor_SMD:C_1206_3216Metric, F.Cu at (111.4, 124.5)
- added C21: 100nF, Capacitor_SMD:C_0805_2012Metric, B.Cu at (116.2, 130.2)
- added C22: 100nF, Capacitor_SMD:C_1206_3216Metric, F.Cu at (107.3, 124.7)
- added C23: 100nF, Capacitor_SMD:C_0805_2012Metric, B.Cu at (110.9, 130.2)
- added C24: 100nF, Capacitor_SMD:C_1206_3216Metric, F.Cu at (103.4, 124.7)
- added C25: 100nF, Capacitor_SMD:C_0805_2012Metric, B.Cu at (105.6, 130.1)
- added C26: 100nF, Capacitor_SMD:C_1206_3216Metric, F.Cu at (99.4, 124.7)
- added C27: 100nF, Capacitor_SMD:C_0805_2012Metric, B.Cu at (100.6, 130.2)
- added C28: 100nF, Capacitor_SMD:C_1206_3216Metric, F.Cu at (95.3, 124.7)
- added C29: 100nF, Capacitor_SMD:C_0805_2012Metric, B.Cu at (95.6, 130.2)
- added C30: 100nF, Capacitor_SMD:C_1206_3216Metric, F.Cu at (91.3, 124.7)
- added C31: 100nF, Capacitor_SMD:C_0805_2012Metric, B.Cu at (90.3, 130.2)
- added C32: 100nF, Capacitor_SMD:C_1206_3216Metric, F.Cu at (87.4, 124.7)
- added C33: 100nF, Capacitor_SMD:C_0805_2012Metric, B.Cu at (84.8, 130.2)
- added C34: 100nF, Capacitor_SMD:C_1206_3216Metric, F.Cu at (83.3, 124.7)
- added C35: 100nF, Capacitor_SMD:C_0805_2012Metric, B.Cu at (169.8, 169.2)
- added C36: 100nF, Capacitor_SMD:C_0805_2012Metric, B.Cu at (45.6, 132.1)
- added C37: 100nF, Capacitor_SMD:C_0805_2012Metric, B.Cu at (44.6, 134.8)
- added C38: 1uF, Capacitor_SMD:C_0805_2012Metric, B.Cu at (43.6, 132.1)
- added C39: 100nF, Capacitor_SMD:C_0805_2012Metric, B.Cu at (39.6, 132.1)
- added C40: 100nF, Capacitor_SMD:C_0805_2012Metric, B.Cu at (38.6, 134.8)
- added C41: 1uF, Capacitor_SMD:C_0805_2012Metric, B.Cu at (37.6, 132.1)
- added C42: 100nF, Capacitor_SMD:C_0805_2012Metric, B.Cu at (77.9, 162.7)
- added C43: 1uF, Capacitor_SMD:C_0805_2012Metric, B.Cu at (77.9, 164.7)
- added C44: 100nF, Capacitor_SMD:C_0805_2012Metric, B.Cu at (84.3, 162.7)
- added C45: 1uF, Capacitor_SMD:C_0805_2012Metric, B.Cu at (84.3, 164.7)
- added C46: 100nF, Capacitor_SMD:C_0805_2012Metric, B.Cu at (91.0, 162.7)
- added C47: 1uF, Capacitor_SMD:C_0805_2012Metric, B.Cu at (91.0, 164.7)
- added C48: 100nF, Capacitor_SMD:C_0805_2012Metric, B.Cu at (97.7, 162.7)
- added C49: 1uF, Capacitor_SMD:C_0805_2012Metric, B.Cu at (97.7, 164.7)
- added C50: 100nF, Capacitor_SMD:C_0805_2012Metric, B.Cu at (104.3, 162.7)
- added C51: 1uF, Capacitor_SMD:C_0805_2012Metric, B.Cu at (104.3, 164.7)
- added C52: 100nF, Capacitor_SMD:C_0805_2012Metric, B.Cu at (111.0, 162.7)
- added C53: 1uF, Capacitor_SMD:C_0805_2012Metric, B.Cu at (111.0, 164.7)
- added C54: 100nF, Capacitor_SMD:C_0805_2012Metric, B.Cu at (117.7, 162.7)
- added C55: 1uF, Capacitor_SMD:C_0805_2012Metric, B.Cu at (117.7, 164.7)
- added C56: 100nF, Capacitor_SMD:C_0805_2012Metric, B.Cu at (124.4, 162.7)
- added C57: 1uF, Capacitor_SMD:C_0805_2012Metric, B.Cu at (124.4, 164.7)
- added COUT3: 100 µF, Capacitor_SMD:C_1210_3225Metric, F.Cu at (162.4, 171.8)
- added D18: 1N4148WS, Diode_SMD:D_SOD-323, F.Cu at (108.1, 128.3)
- added D19: SMBJ33A, Diode_SMD:D_SMA, B.Cu at (99.3, 114.9)
- added D20: 1N4148WS, Diode_SMD:D_SOD-323, F.Cu at (104.0, 128.3)
- added D21: SMBJ33A, Diode_SMD:D_SMA, B.Cu at (95.8, 114.9)
- added D22: 1N4148WS, Diode_SMD:D_SOD-323, F.Cu at (99.8, 128.3)
- added D23: SMBJ33A, Diode_SMD:D_SMA, B.Cu at (92.2, 114.9)
- added D24: 1N4148WS, Diode_SMD:D_SOD-323, F.Cu at (95.7, 128.3)
- added D25: SMBJ33A, Diode_SMD:D_SMA, B.Cu at (88.6, 114.9)
- added D26: 1N4148WS, Diode_SMD:D_SOD-323, F.Cu at (91.6, 128.3)
- added D27: SMBJ33A, Diode_SMD:D_SMA, B.Cu at (85.0, 114.9)
- added D28: 1N4148WS, Diode_SMD:D_SOD-323, F.Cu at (87.5, 128.3)
- added D29: D_Zener_Small, Diode_SMD:D_SOD-123, B.Cu at (158.8, 179.5)
- added D30: ~, Diode_SMD:D_SMB, B.Cu at (168.0, 192.4)
- added D31: SMBJ33A, Diode_SMD:D_SMA, B.Cu at (39.3, 114.9)
- added D32: 1N4148WS, Diode_SMD:D_SOD-323, F.Cu at (48.9, 130.2)
- added D33: SMBJ33A, Diode_SMD:D_SMA, B.Cu at (35.8, 114.9)
- added D34: 1N4148WS, Diode_SMD:D_SOD-323, F.Cu at (42.8, 130.2)
- added D35: SS34, Diode_SMD:D_SMA, B.Cu at (32.0, 192.0)
- added D36: SS34, Diode_SMD:D_SMA, B.Cu at (35.5, 192.0)
- added D37: SS34, Diode_SMD:D_SMA, B.Cu at (39.0, 192.0)
- added D38: SS34, Diode_SMD:D_SMA, B.Cu at (42.6, 192.0)
- added D39: SS34, Diode_SMD:D_SMA, B.Cu at (46.1, 192.0)
- added D40: SS34, Diode_SMD:D_SMA, B.Cu at (49.7, 192.0)
- added D41: SS34, Diode_SMD:D_SMA, B.Cu at (53.3, 192.0)
- added D42: SS34, Diode_SMD:D_SMA, B.Cu at (56.8, 192.0)
- added D43: SS34, Diode_SMD:D_SMA, B.Cu at (84.9, 192.2)
- added D44: SS34, Diode_SMD:D_SMA, B.Cu at (88.4, 192.2)
- added D45: SS34, Diode_SMD:D_SMA, B.Cu at (92.0, 192.2)
- added D46: SS34, Diode_SMD:D_SMA, B.Cu at (95.5, 192.2)
- added D47: SS34, Diode_SMD:D_SMA, B.Cu at (99.0, 192.2)
- added D48: SS34, Diode_SMD:D_SMA, B.Cu at (102.6, 192.2)
- added D49: SS34, Diode_SMD:D_SMA, B.Cu at (106.1, 192.2)
- added D50: SS34, Diode_SMD:D_SMA, B.Cu at (109.7, 192.2)
- added H1: MountingHole, MountingHole:MountingHole_3.2mm_M3_Pad, F.Cu at (26.5, 130.3)
- added H2: MountingHole, MountingHole:MountingHole_3.2mm_M3_Pad, F.Cu at (168.5, 130.3)
- added H3: MountingHole, MountingHole:MountingHole_3.2mm_M3_Pad, F.Cu at (168.5, 176.6)
- added H4: MountingHole, MountingHole:MountingHole_3.2mm_M3_Pad, F.Cu at (26.5, 176.6)
- added H5: MountingHole, MountingHole:MountingHole_3.2mm_M3_Pad, F.Cu at (51.9, 38.8)
- added H6: MountingHole, MountingHole:MountingHole_3.2mm_M3_Pad, F.Cu at (51.9, 85.1)
- added H7: MountingHole, MountingHole:MountingHole_3.2mm_M3_Pad, F.Cu at (193.9, 38.8)
- added H8: MountingHole, MountingHole:MountingHole_3.2mm_M3_Pad, F.Cu at (193.9, 85.1)
- added J13: Conn_02x20_Counter_Clockwise, Connector_IDC:IDC-Header_2x20_P2.54mm_Vertical, B.Cu at (54.1, 50.8)
- added J14: DI_IN_Connector, Connector_Phoenix_MC:PhoenixContact_MC_1,5_2-G-3.5_1x02_P3.50mm_Horizontal, F.Cu at (166.3, 187.9)
- added J2: Conn_02x20_Counter_Clockwise, Connector_IDC:IDC-Header_2x20_P2.54mm_Vertical, F.Cu at (28.4, 153.6)
- added J3: Conn_02x20_Counter_Clockwise, Connector_IDC:IDC-Header_2x08_P2.54mm_Vertical, F.Cu at (243.6, 26.9)
- added J6: Conn_02x20_Counter_Clockwise, Connector_IDC:IDC-Header_2x06_P2.54mm_Vertical, B.Cu at (151.4, 36.9)
- added J8: DI_IN_Connector, Connector_Phoenix_MC:PhoenixContact_MC_1,5_9-G-3.5_1x09_P3.50mm_Horizontal, F.Cu at (131.2, 187.9)
- added J9: Conn_02x20_Counter_Clockwise, Connector_IDC:IDC-Header_2x08_P2.54mm_Vertical, F.Cu at (133.6, 133.8)
- added MOD1: ~, MyModules:WeAct_STM32H743VIT6, F.Cu at (56.4, 73.7)
- added Q10: NMOS AOD4184A, Package_TO_SOT_THT:TO-220-3_Vertical, F.Cu at (75.6, 172.6)
- added Q11: NMOS AOD4184A, Package_TO_SOT_THT:TO-220-3_Vertical, F.Cu at (82.0, 172.6)
- added Q12: NMOS AOD4184A, Package_TO_SOT_THT:TO-220-3_Vertical, F.Cu at (88.7, 172.6)
- added Q13: NMOS AOD4184A, Package_TO_SOT_THT:TO-220-3_Vertical, F.Cu at (95.3, 172.6)
- added Q14: NMOS AOD4184A, Package_TO_SOT_THT:TO-220-3_Vertical, F.Cu at (102.0, 172.6)
- added Q15: NMOS AOD4184A, Package_TO_SOT_THT:TO-220-3_Vertical, F.Cu at (108.7, 172.6)
- added Q16: NMOS AOD4184A, Package_TO_SOT_THT:TO-220-3_Vertical, F.Cu at (115.4, 172.6)
- added Q17: NMOS AOD4184A, Package_TO_SOT_THT:TO-220-3_Vertical, F.Cu at (122.1, 172.6)
- added R100: 10 Ω, Resistor_SMD:R_1206_3216Metric, B.Cu at (116.5, 167.5)
- added R101: 4.7Ω, Resistor_SMD:R_1206_3216Metric, B.Cu at (116.5, 169.8)
- added R102: 4.7k, Resistor_SMD:R_1206_3216Metric, B.Cu at (117.7, 173.7)
- added R103: 47Ω, Resistor_SMD:R_1206_3216Metric, F.Cu at (122.5, 165.1)
- added R104: 10 Ω, Resistor_SMD:R_1206_3216Metric, B.Cu at (123.2, 167.5)
- added R105: 4.7Ω, Resistor_SMD:R_1206_3216Metric, B.Cu at (123.2, 169.8)
- added R106: 4.7k, Resistor_SMD:R_1206_3216Metric, B.Cu at (124.4, 173.7)
- added R43: 6.8k, Resistor_SMD:R_1206_3216Metric, B.Cu at (91.9, 124.9)
- added R44: 4.7k, Resistor_SMD:R_0805_2012Metric, B.Cu at (96.2, 139.8)
- added R45: 220Ω, Resistor_SMD:R_0805_2012Metric, B.Cu at (90.8, 135.7)
- added R46: 6.8k, Resistor_SMD:R_1206_3216Metric, B.Cu at (84.9, 124.9)
- added R47: 6.8k, Resistor_SMD:R_1206_3216Metric, B.Cu at (87.2, 124.9)
- added R48: 4.7k, Resistor_SMD:R_0805_2012Metric, B.Cu at (91.8, 139.8)
- added R49: 220Ω, Resistor_SMD:R_0805_2012Metric, B.Cu at (85.3, 135.7)
- added R50: 6.8k, Resistor_SMD:R_1206_3216Metric, B.Cu at (82.5, 124.9)
- added R51: 6.8k, Resistor_SMD:R_1206_3216Metric, B.Cu at (80.2, 124.9)
- added R52: 4.7k, Resistor_SMD:R_0805_2012Metric, B.Cu at (87.2, 139.8)
- added R53: 100k, Resistor_SMD:R_1206_3216Metric, B.Cu at (163.8, 179.4)
- added R54: 100k, Resistor_SMD:R_1206_3216Metric, B.Cu at (161.4, 179.4)
- added R55: 2k2, Resistor_SMD:R_1206_3216Metric, B.Cu at (39.4, 122.4)
- added R56: 2k2, Resistor_SMD:R_1206_3216Metric, B.Cu at (40.8, 127.4)
- added R57: 1k, Resistor_SMD:R_0805_2012Metric, F.Cu at (49.4, 139.6)
- added R58: 2k2, Resistor_SMD:R_1206_3216Metric, B.Cu at (35.9, 122.4)
- added R59: 2k2, Resistor_SMD:R_1206_3216Metric, B.Cu at (37.3, 127.4)
- added R60: 1k, Resistor_SMD:R_0805_2012Metric, F.Cu at (43.4, 139.6)
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Connections:
- C1 pad 1: /DI_Channel/DI_FIELD_FILT -> +5V
- C1 pad 2: FIELD_GND -> Logic_GND
- C2 pad 1: /DI_Channel1/DI_FIELD_FILT -> +3V3
- C2 pad 2: FIELD_GND -> Logic_GND
- C3 pad 1: /DI_Channel2/DI_FIELD_FILT -> +5V
- C3 pad 2: FIELD_GND -> Logic_GND
- C4 pad 1: /DI_Channel3/DI_FIELD_FILT -> +5V
- C4 pad 2: FIELD_GND -> Logic_GND
- C5 pad 1: /DI_Channel4/DI_FIELD_FILT -> +3V3
- C5 pad 2: FIELD_GND -> Logic_GND
- C6 pad 1: /DI_Channel5/DI_FIELD_FILT -> +5V
- C6 pad 2: FIELD_GND -> Logic_GND
- C7 pad 1: /DI_Channel6/DI_FIELD_FILT -> +5V
- C7 pad 2: FIELD_GND -> Logic_GND
- C8 pad 1: /DI_Channel7/DI_FIELD_FILT -> +3V3
- C8 pad 2: FIELD_GND -> Logic_GND
- C9 pad 1: Net-(U17-CB) -> +5V
- C9 pad 2: Net-(U17-SW) -> Logic_GND
- CCOUT1 pad 1: +3.3V -> 3V3_LOGIC
- CCOUT1 pad 2: LOGIC_GND -> GND
- CCOUT2 pad 1: +3.3V -> 3V3_LOGIC
- CCOUT2 pad 2: LOGIC_GND -> GND
- CIN1 pad 2: FIELD_GND -> GND
- CIN2 pad 2: FIELD_GND -> GND
- CIN3 pad 2: FIELD_GND -> GND
- CIN4 pad 1: +5V -> 5V_MAIN
- CIN4 pad 2: LOGIC_GND -> GND
- CIN5 pad 1: +5V -> 5V_MAIN
- CIN5 pad 2: LOGIC_GND -> GND
- COUT1 pad 1: +5V -> 5V_MAIN
- COUT1 pad 2: LOGIC_GND -> GND
- COUT2 pad 1: +5V -> 5V_MAIN
- COUT2 pad 2: LOGIC_GND -> GND
- D1 pad 1: /DI_Channel/DI_FIELD_IN -> /DI_IN9
- D1 pad 2: FIELD_GND -> Field_GND
- D10 pad 1: /DO_Channel1/DO_OUT -> Net-(D10-K)
- D10 pad 2: +24V -> Field_GND
- D11 pad 1: /DO_Channel2/DO_OUT -> /DI_IN13
- D11 pad 2: +24V -> Field_GND
- D12 pad 1: /DO_Channel3/DO_OUT -> Net-(D12-K)
- D12 pad 2: +24V -> Field_GND
- D13 pad 1: /DO_Channel4/DO_OUT -> /DI_IN1
- D13 pad 2: +24V -> Field_GND
- D14 pad 1: /DO_Channel5/DO_OUT -> Net-(D14-K)
- D14 pad 2: +24V -> Field_GND
- D15 pad 1: /DO_Channel6/DO_OUT -> /DI_IN2
- D15 pad 2: +24V -> Field_GND
- D16 pad 1: /DO_Channel7/DO_OUT -> Net-(D16-K)
- D16 pad 2: +24V -> Field_GND
- D17 pad 1: Net-(D17-A1) -> /DI_IN3
- D17 pad 2: FIELD_GND -> Field_GND
- D2 pad 1: /DI_Channel1/DI_FIELD_IN -> Net-(D2-K)
- D2 pad 2: FIELD_GND -> Field_GND
- D3 pad 1: /DI_Channel2/DI_FIELD_IN -> /DI_IN10
- D3 pad 2: FIELD_GND -> Field_GND
- D4 pad 1: /DI_Channel3/DI_FIELD_IN -> Net-(D4-K)
- D4 pad 2: FIELD_GND -> Field_GND
- D5 pad 1: /DI_Channel4/DI_FIELD_IN -> /DI_IN16
- D5 pad 2: FIELD_GND -> Field_GND
- D6 pad 1: /DI_Channel5/DI_FIELD_IN -> Net-(D6-K)
- D6 pad 2: FIELD_GND -> Field_GND
- D7 pad 1: /DI_Channel6/DI_FIELD_IN -> /DI_IN11
- D7 pad 2: FIELD_GND -> Field_GND
- D8 pad 1: /DI_Channel7/DI_FIELD_IN -> Net-(D8-K)
- D8 pad 2: FIELD_GND -> Field_GND
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Routing:
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- removed copper zone on F.Cu, net +3.3V
- removed copper zone on B.Cu, net FIELD_GND
- removed copper zone on F.Cu, net FIELD_GND
- removed copper zone on F.Cu, net LOGIC_GND
Other:
- board size 230 x 90 mm -> 175.3 x 163.3 mm

Commit message: 112
Parts:
- removed the C39 at (39.6, 132.1)
- removed the C40 at (38.6, 134.8)
- removed the C41 at (37.6, 132.1)
- removed the C7 at (33.6, 132.1)
- removed the C8 at (32.5, 134.8)
- removed the C9 at (31.6, 132.1)
- removed the D27 at (85.0, 114.9)
- removed the D33 at (35.8, 114.9)
- removed the D34 at (42.8, 130.2)
- removed the D5 at (32.2, 114.9)
- removed the D6 at (36.8, 130.2)
- removed J13: Conn_02x20_Counter_Clockwise, Connector_IDC:IDC-Header_2x20_P2.54mm_Vertical
- removed the J3 at (243.6, 26.9)
- removed the J6 at (151.4, 36.9)
- removed the R10 at (33.8, 127.4)
- removed the R11 at (37.4, 139.6)
- removed the R58 at (35.9, 122.4)
- removed the R59 at (37.3, 127.4)
- removed the R60 at (43.4, 139.6)
- removed the R9 at (32.4, 122.4)
- removed the U2 at (243.3, 62.6)
- removed the U35 at (38.8, 138.5)
- removed the U36 at (43.1, 134.8)
- removed the U7 at (32.7, 138.5)
- removed the U8 at (37.0, 134.8)
- added D19: SMBJ33A, Diode_SMD:D_SMA, B.Cu at (60.7, 114.9)
- added U6: ~, MyModules:DAC8568_Module_57x52mm, F.Cu at (136.5, 90.8)
- J10: value DI_IN_Connector -> Conn_02x20_Counter_Clockwise; footprint Connector_Phoenix_MC:PhoenixContact_MC_1,5_12-G-3.5_1x12_P3.50mm_Horizontal -> Connector_IDC:IDC-Header_2x25_P2.54mm_Vertical; moved to B.Cu
- J2: footprint Connector_IDC:IDC-Header_2x20_P2.54mm_Vertical -> Connector_IDC:IDC-Header_2x25_P2.54mm_Vertical
- J4: value Conn_02x20_Counter_Clockwise -> Conn_02x08_Counter_Clockwise; footprint Connector_IDC:IDC-Header_2x08_P2.54mm_Vertical -> Connector_PinSocket_2.54mm:PinSocket_2x08_P2.54mm_Vertical_SMD
- J7: value Conn_02x20_Counter_Clockwise -> DI_IN_Connector; footprint Connector_IDC:IDC-Header_2x06_P2.54mm_Vertical -> Connector_Phoenix_MC:PhoenixContact_MC_1,5_12-G-3.5_1x12_P3.50mm_Horizontal
- J8: footprint Connector_Phoenix_MC:PhoenixContact_MC_1,5_9-G-3.5_1x09_P3.50mm_Horizontal -> Connector_Phoenix_MC:PhoenixContact_MC_1,5_12-G-3.5_1x12_P3.50mm_Horizontal
- J9: value Conn_02x20_Counter_Clockwise -> Conn_01x05; footprint Connector_IDC:IDC-Header_2x08_P2.54mm_Vertical -> Connector_PinHeader_2.54mm:PinHeader_1x07_P2.54mm_Vertical
- U1: footprint MyModules:DAC8568_Module_57x52mm -> MyModules:AD7606_Module_40x30mm
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- renumbered C13 to C10, C14 to C11, C15 to C12, C16 to C13, C17 to C14, C18 to C15, C19 to C16, C20 to C17, C21 to C18, C22 to C19, C23 to C20, C24 to C21, C25 to C22, C26 to C23, C27 to C24, C28 to C25, C29 to C26, C30 to C27, C31 to C28, C32 to C29, C33 to C30, C34 to C31, C35 to C32, C36 to C33, C37 to C34, C38 to C35, C42 to C36, C43 to C37, C44 to C38, C45 to C39, C46 to C40, C47 to C41, C48 to C42, C49 to C43, C50 to C44, C51 to C45, C52 to C46, C53 to C47, C54 to C48, C55 to C49, C56 to C50, C57 to C51, C10 to C7, C11 to C8, C12 to C9, D12 to D10, D13 to D11, D14 to D12, D15 to D13, D16 to D14, D17 to D15, D18 to D16, D19 to D17, D20 to D18, D22 to D20, D24 to D22, D26 to D24, D28 to D26, D29 to D27, D30 to D28, D31 to D29, D32 to D30, D35 to D31, D36 to D32, D37 to D33, D38 to D34, D39 to D35, D40 to D36, D41 to D37, D42 to D38, D43 to D39, D44 to D40, D45 to D41, D46 to D42, D47 to D43, D48 to D44, D49 to D45, D50 to D46, D7 to D5, D8 to D6, D9 to D7, D10 to D8, D11 to D9, J14 to J11, J5 to J3, J11 to J5, J12 to J6, R13 to R10, R106 to R100, R14 to R11, R15 to R12, R16 to R13, R17 to R14, R18 to R15, R19 to R16, R20 to R17, R21 to R18, R22 to R19, R23 to R20, R24 to R21, R25 to R22, R26 to R23, R27 to R24, R28 to R25, R29 to R26, R30 to R27, R31 to R28, R32 to R29, R33 to R30, R34 to R31, R35 to R32, R36 to R33, R37 to R34, R38 to R35, R39 to R36, R40 to R37, R41 to R38, R42 to R39, R43 to R40, R44 to R41, R45 to R42, R46 to R43, R47 to R44, R48 to R45, R49 to R46, R50 to R47, R51 to R48, R52 to R49, R53 to R50, R54 to R51, R55 to R52, R56 to R53, R57 to R54, R61 to R55, R62 to R56, R63 to R57, R64 to R58, R65 to R59, R66 to R60, R67 to R61, R68 to R62, R69 to R63, R70 to R64, R71 to R65, R72 to R66, R73 to R67, R74 to R68, R75 to R69, R76 to R70, R77 to R71, R78 to R72, R79 to R73, R80 to R74, R81 to R75, R82 to R76, R83 to R77, R84 to R78, R85 to R79, R86 to R80, R87 to R81, R88 to R82, R89 to R83, R90 to R84, R91 to R85, R92 to R86, R93 to R87, R94 to R88, R95 to R89, R12 to R9, R96 to R90, R97 to R91, R98 to R92, R99 to R93, R100 to R94, R101 to R95, R102 to R96, R103 to R97, R104 to R98, R105 to R99, U12 to U10, U13 to U11, U14 to U12, U15 to U13, U16 to U14, U17 to U15, U18 to U16, U19 to U17, U20 to U18, U21 to U19, U3 to U2, U22 to U20, U23 to U21, U24 to U22, U25 to U23, U26 to U24, U27 to U25, U28 to U26, U29 to U27, U30 to U28, U31 to U29, U4 to U3, U32 to U30, U33 to U31, U34 to U32, U37 to U33, U38 to U34, U39 to U35, U40 to U36, U41 to U37, U42 to U38, U43 to U39, U5 to U4, U44 to U40, U6 to U5, U9 to U7, U10 to U8, U11 to U9
Connections:
- D21 pad 1: /DI_IN5 -> /DI_IN6
- D23 pad 1: /DI_IN6 -> /DI_IN7
- D25 pad 1: /DI_IN7 -> /DI_IN8
- J1 pad 1: Field_GND -> unconnected-(J1-Pin_1-Pad1)
- J1 pad 10: /DI_IN8 -> /DI_IN1
- J1 pad 11: Field_GND -> /DI_IN2
- J1 pad 12: Field_GND -> /DI_IN3
- J1 pad 2: Field_GND -> /AD7606_V8
- J1 pad 3: /DI_IN1 -> /AD7606_V7
- J1 pad 4: /DI_IN2 -> /AD7606_V6
- J1 pad 5: /DI_IN3 -> /AD7606_V5
- J1 pad 6: /DI_IN4 -> /AD7606_V4
- J1 pad 7: /DI_IN5 -> /AD7606_V3
- J1 pad 8: /DI_IN6 -> /AD7606_V2
- J1 pad 9: /DI_IN7 -> /AD7606_V1
- J10 pad 1: unconnected-(J10-Pin_1-Pad1) -> /MCU_STM32/DO_SLOW_CTRL1
- J10 pad 10: unconnected-(J10-Pin_10-Pad10) -> /MCU_STM32/DI_IN9_LOGIC12
- J10 pad 11: unconnected-(J10-Pin_11-Pad11) -> /MCU_STM32/DO_SLOW_CTRL6
- J10 pad 12: unconnected-(J10-Pin_12-Pad12) -> /MCU_STM32/DI_IN9_LOGIC11
- J10 pad 2: unconnected-(J10-Pin_2-Pad2) -> Logic_GND
- J10 pad 3: unconnected-(J10-Pin_3-Pad3) -> /MCU_STM32/DO_SLOW_CTRL2
- J10 pad 4: unconnected-(J10-Pin_4-Pad4) -> Logic_GND
- J10 pad 5: unconnected-(J10-Pin_5-Pad5) -> /MCU_STM32/DO_SLOW_CTRL3
- J10 pad 6: unconnected-(J10-Pin_6-Pad6) -> /MCU_STM32/DI_IN9_LOGIC14
- J10 pad 7: unconnected-(J10-Pin_7-Pad7) -> /MCU_STM32/DO_SLOW_CTRL4
- J10 pad 8: unconnected-(J10-Pin_8-Pad8) -> /MCU_STM32/DI_IN9_LOGIC13
- J10 pad 9: unconnected-(J10-Pin_9-Pad9) -> /MCU_STM32/DO_SLOW_CTRL5
- J2 pad 17: /DO_PWM_CTRL1 -> Logic_GND
- J2 pad 18: /DI_SLOW_LOGIC8 -> Logic_GND
- J2 pad 19: /DO_PWM_CTRL2 -> Logic_GND
- J2 pad 2: /DI_IN9_LOGIC16 -> Logic_GND
- J2 pad 20: /DI_SLOW_LOGIC7 -> Logic_GND
- J2 pad 21: /DO_PWM_CTRL3 -> Logic_GND
- J2 pad 22: /DI_SLOW_LOGIC6 -> Logic_GND
- J2 pad 23: /DO_PWM_CTRL4 -> Logic_GND
- J2 pad 24: /DI_SLOW_LOGIC5 -> Logic_GND
- J2 pad 25: /DO_PWM_CTRL5 -> /DO_PWM_CTRL1
- J2 pad 26: /DI_SLOW_LOGIC4 -> /DI_SLOW_LOGIC8
- J2 pad 27: /DO_PWM_CTRL6 -> /DO_PWM_CTRL2
- J2 pad 28: /DI_SLOW_LOGIC3 -> /DI_SLOW_LOGIC7
- J2 pad 29: /DO_PWM_CTRL7 -> /DO_PWM_CTRL3
- J2 pad 30: /DI_SLOW_LOGIC2 -> /DI_SLOW_LOGIC6
- J2 pad 31: /DO_PWM_CTRL8 -> /DO_PWM_CTRL4
- J2 pad 32: /DI_SLOW_LOGIC1 -> /DI_SLOW_LOGIC5
- J2 pad 33: unconnected-(J2-Pin_33-Pad33) -> /DO_PWM_CTRL5
- J2 pad 34: unconnected-(J2-Pin_34-Pad34) -> /DI_SLOW_LOGIC4
- J2 pad 35: unconnected-(J2-Pin_35-Pad35) -> /DO_PWM_CTRL6
- J2 pad 36: unconnected-(J2-Pin_36-Pad36) -> /DI_SLOW_LOGIC3
- J2 pad 37: unconnected-(J2-Pin_37-Pad37) -> /DO_PWM_CTRL7
- J2 pad 38: unconnected-(J2-Pin_38-Pad38) -> /DI_SLOW_LOGIC2
- J2 pad 39: unconnected-(J2-Pin_39-Pad39) -> /DO_PWM_CTRL8
- J2 pad 4: /DI_IN9_LOGIC15 -> Logic_GND
- J2 pad 40: unconnected-(J2-Pin_40-Pad40) -> /DI_SLOW_LOGIC1
- J6 pad 1: Field_GND -> /DI_IN4
- J6 pad 10: /DI_IN16 -> /DI_IN13
- J6 pad 11: Field_GND -> /DI_IN14
- J6 pad 2: Field_GND -> /DI_IN5
- J6 pad 3: /DI_IN9 -> /DI_IN6
- J6 pad 4: /DI_IN10 -> /DI_IN7
- J6 pad 5: /DI_IN11 -> /DI_IN8
- J6 pad 6: /DI_IN12 -> /DI_IN9
- J6 pad 7: /DI_IN13 -> /DI_IN10
- J6 pad 8: /DI_IN14 -> /DI_IN11
- J6 pad 9: /DI_IN15 -> /DI_IN12
- J7 pad 1: Field_GND -> unconnected-(J7-Pin_1-Pad1)
- J7 pad 10: Net-(J7-Pin_10) -> unconnected-(J7-Pin_10-Pad10)
- J7 pad 11: Net-(J7-Pin_11) -> unconnected-(J7-Pin_11-Pad11)
- J7 pad 12: Net-(J7-Pin_12) -> unconnected-(J7-Pin_12-Pad12)
- J7 pad 2: Net-(J7-Pin_2) -> unconnected-(J7-Pin_2-Pad2)
- J7 pad 3: Field_GND -> unconnected-(J7-Pin_3-Pad3)
- J7 pad 4: Net-(J7-Pin_4) -> unconnected-(J7-Pin_4-Pad4)
- J7 pad 5: Field_GND -> unconnected-(J7-Pin_5-Pad5)
- J7 pad 6: Net-(J7-Pin_6) -> unconnected-(J7-Pin_6-Pad6)
- J7 pad 7: Field_GND -> unconnected-(J7-Pin_7-Pad7)
- J7 pad 8: Net-(J7-Pin_8) -> unconnected-(J7-Pin_8-Pad8)
- J7 pad 9: Net-(J7-Pin_9) -> unconnected-(J7-Pin_9-Pad9)
- J8 pad 1: Net-(J7-Pin_9) -> unconnected-(J8-Pin_1-Pad1)
- J8 pad 2: Net-(J7-Pin_11) -> unconnected-(J8-Pin_2-Pad2)
- J8 pad 3: Net-(J7-Pin_12) -> unconnected-(J8-Pin_3-Pad3)
- J8 pad 4: Net-(J7-Pin_10) -> unconnected-(J8-Pin_4-Pad4)
- J8 pad 5: Net-(J7-Pin_8) -> unconnected-(J8-Pin_5-Pad5)
- J8 pad 6: Net-(J7-Pin_6) -> unconnected-(J8-Pin_6-Pad6)
- J8 pad 7: Net-(J7-Pin_4) -> unconnected-(J8-Pin_7-Pad7)
- J8 pad 8: Net-(J7-Pin_2) -> unconnected-(J8-Pin_8-Pad8)
- J8 pad 9: Field_GND -> unconnected-(J8-Pin_9-Pad9)
- J9 pad 1: unconnected-(J9-Pin_1-Pad1) -> /MCU_STM32/DAC8568_SCLK
- J9 pad 2: unconnected-(J9-Pin_2-Pad2) -> /MCU_STM32/DAC8568_DIN
- J9 pad 3: unconnected-(J9-Pin_3-Pad3) -> /MCU_STM32/DAC8568_CLR
- J9 pad 4: unconnected-(J9-Pin_4-Pad4) -> /MCU_STM32/DAC8568_SYNC
- J9 pad 5: unconnected-(J9-Pin_5-Pad5) -> /MCU_STM32/DAC8568_LDAC
- J9 pad 6: unconnected-(J9-Pin_6-Pad6) -> Logic_GND
- J9 pad 7: unconnected-(J9-Pin_7-Pad7) -> +5V
- MOD1 pad 1: Net-(J13-Pin_1) -> Logic_GND
- MOD1 pad 10: unconnected-(MOD1-B4-Pad10) -> /MCU_STM32/DO_PWM_CTRL1
- MOD1 pad 12: unconnected-(MOD1-D7-Pad12) -> /MCU_STM32/DI_SLOW_LOGIC8
- MOD1 pad 13: unconnected-(MOD1-D6-Pad13) -> /MCU_STM32/DI_SLOW_LOGIC7
- MOD1 pad 14: unconnected-(MOD1-D5-Pad14) -> /MCU_STM32/DI_SLOW_LOGIC6
- MOD1 pad 15: unconnected-(MOD1-D4-Pad15) -> /MCU_STM32/DI_SLOW_LOGIC5
- MOD1 pad 16: unconnected-(MOD1-D3-Pad16) -> /MCU_STM32/DI_SLOW_LOGIC4
- MOD1 pad 17: unconnected-(MOD1-D2-Pad17) -> /MCU_STM32/DI_SLOW_LOGIC3
- MOD1 pad 18: unconnected-(MOD1-D1-Pad18) -> /MCU_STM32/DI_SLOW_LOGIC2
- MOD1 pad 19: unconnected-(MOD1-D0-Pad19) -> /MCU_STM32/DI_SLOW_LOGIC1
- MOD1 pad 2: Net-(J13-Pin_3) -> unconnected-(MOD1-+5V-Pad2)
- MOD1 pad 23: unconnected-(MOD1-A15-Pad23) -> /MCU_STM32/DI_IN9_LOGIC14
- MOD1 pad 27: unconnected-(MOD1-A9-Pad27) -> /MCU_STM32/DAC8568_SCLK
- MOD1 pad 3: unconnected-(MOD1-E1-Pad3) -> /MCU_STM32/DO_SLOW_CTRL2
- MOD1 pad 31: unconnected-(MOD1-C7-Pad31) -> /MCU_STM32/DI_IN9_LOGIC9
- MOD1 pad 32: unconnected-(MOD1-C6-Pad32) -> /MCU_STM32/DI_IN9_LOGIC10
- MOD1 pad 34: unconnected-(MOD1-D14-Pad34) -> /MCU_STM32/DO_PWM_CTRL8
- MOD1 pad 35: unconnected-(MOD1-D13-Pad35) -> /MCU_STM32/DO_PWM_CTRL7
- MOD1 pad 36: unconnected-(MOD1-D12-Pad36) -> /MCU_STM32/DO_PWM_CTRL2
- MOD1 pad 38: unconnected-(MOD1-D10-Pad38) -> /MCU_STM32/DO_SLOW_CTRL8
- MOD1 pad 4: unconnected-(MOD1-E0-Pad4) -> /MCU_STM32/DO_SLOW_CTRL1
- MOD1 pad 40: unconnected-(MOD1-D8-Pad40) -> /MCU_STM32/DAC8568_SYNC
- MOD1 pad 41: unconnected-(MOD1-B15-Pad41) -> /MCU_STM32/DAC8568_LDAC
- MOD1 pad 42: unconnected-(MOD1-B14-Pad42) -> /MCU_STM32/DO_PWM_CTRL3
- MOD1 pad 45: unconnected-(MOD1-GND-Pad45) -> Logic_GND
- MOD1 pad 47: unconnected-(MOD1-E2-Pad47) -> /MCU_STM32/DO_SLOW_CTRL3
- MOD1 pad 48: unconnected-(MOD1-E3-Pad48) -> /MCU_STM32/DO_SLOW_CTRL4
- MOD1 pad 49: unconnected-(MOD1-E4-Pad49) -> /MCU_STM32/DO_SLOW_CTRL5
- MOD1 pad 5: unconnected-(MOD1-B9-Pad5) -> /MCU_STM32/DO_PWM_CTRL6
- MOD1 pad 50: unconnected-(MOD1-E5-Pad50) -> /MCU_STM32/DO_SLOW_CTRL6
- MOD1 pad 51: unconnected-(MOD1-E6-Pad51) -> /MCU_STM32/DO_SLOW_CTRL7
- MOD1 pad 58: unconnected-(MOD1-C3-Pad58) -> /MCU_STM32/DAC8568_DIN
- MOD1 pad 59: unconnected-(MOD1-GND-Pad59) -> Logic_GND
- MOD1 pad 6: unconnected-(MOD1-B8-Pad6) -> /MCU_STM32/DO_PWM_CTRL5
- MOD1 pad 61: unconnected-(MOD1-A0-Pad61) -> /MCU_STM32/DI_IN9_LOGIC13
- MOD1 pad 64: unconnected-(MOD1-A3-Pad64) -> /MCU_STM32/DO_PWM_CTRL4
- MOD1 pad 66: unconnected-(MOD1-A5-Pad66) -> /MCU_STM32/AD7606_SCK
- MOD1 pad 67: unconnected-(MOD1-A6-Pad67) -> /MCU_STM32/AD7606_MISO
- MOD1 pad 71: unconnected-(MOD1-B0-Pad71) -> /MCU_STM32/AD7606_CS
- MOD1 pad 74: unconnected-(MOD1-E7-Pad74) -> /MCU_STM32/AD7606_RST
- MOD1 pad 75: unconnected-(MOD1-E8-Pad75) -> /MCU_STM32/AD7606_BUSY
- MOD1 pad 76: unconnected-(MOD1-E9-Pad76) -> /MCU_STM32/DI_IN9_LOGIC12
- MOD1 pad 77: unconnected-(MOD1-E10-Pad77) -> /MCU_STM32/DAC8568_CLR
- MOD1 pad 78: unconnected-(MOD1-E11-Pad78) -> /MCU_STM32/DI_IN9_LOGIC11
- MOD1 pad 87: unconnected-(MOD1-GND-Pad87) -> Logic_GND
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Routing:
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
Commit message: 112
Parts:
- removed H1, H2, H3, H4, H5, H6, H7, H8: MountingHole, MountingHole:MountingHole_3.2mm_M3_Pad
- added J10: Conn_02x07_Counter_Clockwise, Connector_PinSocket_2.54mm:PinSocket_2x07_P2.54mm_Horizontal, F.Cu at (156.9, 36.1)
- added J11: Conn_02x07_Counter_Clockwise, Connector_PinSocket_2.54mm:PinSocket_2x07_P2.54mm_Horizontal, F.Cu at (243.8, 48.4)
- C36, C37, C38, C39, C42, C43, C46, C47, R1, R2, R57, R58, R61, R62, R65, R66, R70, R71, R72, R74, R75, R76, R82, R83, R84, R90, R91, R92: moved to F.Cu
- Q1, Q10, Q11, Q13, Q15, Q4, Q6, Q8: footprint Package_TO_SOT_THT:TO-220-3_Vertical -> Package_TO_SOT_SMD:TO-252-3_TabPin2
- Q12, Q14, Q16, Q17, Q3, Q5, Q7, Q9: footprint Package_TO_SOT_THT:TO-220-3_Vertical -> Package_TO_SOT_SMD:TO-252-3_TabPin2; moved to B.Cu
- R77, R85, R93, R97, U35, U37, U39, U40: moved to B.Cu
- moved J7 70.7 mm to (200.9, 200.2)
- moved Q9 15.2 mm to (53.1, 176.7)
- moved Q7 14.4 mm to (44.2, 176.7)
- moved Q5 14.2 mm to (34.3, 176.7)
- moved Q3 13.3 mm to (26.4, 176.7)
- moved Q8 13.2 mm to (52.9, 176.7)
- moved Q1 13.0 mm to (27.0, 176.7)
- moved Q6 12.9 mm to (44.3, 176.7)
- moved Q4 12.9 mm to (35.7, 176.7)
- moved R96 12.0 mm to (99.4, 168.7), turned to 180 degrees
- moved R88 11.4 mm to (86.7, 168.7), turned to 180 degrees
- moved R95 11.1 mm to (99.4, 164.1), turned to 0 degrees
- moved R68 11.1 mm to (53.5, 167.8), turned to 180 degrees
- moved R80 10.8 mm to (74.0, 168.7), turned to 180 degrees
- moved Q11 10.6 mm to (84.2, 176.7)
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- renumbered J10 to J12, J11 to J13
Connections:
- J2 pad 41: unconnected-(J2-Pin_41-Pad41) -> Logic_GND
- J2 pad 42: unconnected-(J2-Pin_42-Pad42) -> Logic_GND
- J2 pad 43: unconnected-(J2-Pin_43-Pad43) -> Logic_GND
- J2 pad 44: unconnected-(J2-Pin_44-Pad44) -> Logic_GND
- J3 pad 11: +24V -> Field_GND
- J3 pad 12: +24V -> Field_GND
- J5 pad 11: +24V -> Field_GND
- J5 pad 4: /DO_OUT10 -> /DO_OUT11
- J5 pad 5: /DO_OUT11 -> /DO_OUT10
- J5 pad 6: /DO_OUT12 -> /DO_OUT13
- J5 pad 7: /DO_OUT13 -> /DO_OUT12
- J5 pad 8: /DO_OUT14 -> /DO_OUT15
- J5 pad 9: /DO_OUT15 -> /DO_OUT14
Routing:
- net +5V: track 216.5 -> 140.0 mm, vias 16 -> 0
- net /DO_OUT8: track 52.8 -> 11.4 mm
- net /DO_OUT7: track 51.2 -> 10.1 mm
- net /DO_OUT1: track 51.5 -> 12.0 mm
- net /DO_OUT5: track 48.3 -> 10.5 mm
- net /DO_OUT6: track 49.8 -> 12.2 mm
- net /DO_OUT3: track 48.8 -> 11.3 mm
- net /DO_OUT2: track 50.2 -> 13.8 mm
- net /DO_OUT4: track 47.6 -> 13.0 mm
- net /DO_OUT9: track 50.4 -> 22.9 mm
- net /DO_OUT12: track 36.7 -> 11.3 mm
- net /DO_OUT16: track 35.8 -> 11.3 mm
- net /DO_OUT11: track 41.3 -> 17.9 mm
- net /AD7606_CS: track 30.4 -> 53.4 mm
- net /DO_OUT14: track 31.8 -> 9.98 mm
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
Commit message: 112
Parts:
- removed the J11 at (243.8, 48.4)
- removed the J12 at (67.4, 55.9)
- removed the J2 at (28.3, 153.2)
- removed the J4 at (255.1, 123.0)
- added J1: DI_IN_Connector, Connector_Phoenix_MC:PhoenixContact_MC_1,5_2-G-3.5_1x02_P3.50mm_Horizontal, F.Cu at (150.0, 94.3)
- added J14: Conn_02x20_Counter_Clockwise, Connector_PinSocket_2.54mm:PinSocket_2x28_P2.54mm_Vertical, B.Cu at (19.6, 45.8)
- added J15: Conn_02x07_Counter_Clockwise, Connector_PinSocket_2.54mm:PinSocket_2x07_P2.54mm_Vertical, B.Cu at (135.4, 33.0)
- added J3: Conn_02x20_Counter_Clockwise, Connector_PinHeader_2.54mm:PinHeader_2x28_P2.54mm_Vertical, F.Cu at (19.7, 127.7)
- added J5: Conn_02x07_Counter_Clockwise, Connector_PinSocket_2.54mm:PinSocket_2x07_P2.54mm_Horizontal, F.Cu at (121.2, 139.6)
- added J6: Conn_02x07_Counter_Clockwise, Connector_PinSocket_2.54mm:PinSocket_2x07_P2.54mm_Vertical, B.Cu at (144.0, 32.3)
- added J7: Conn_02x07_Counter_Clockwise, Connector_PinSocket_2.54mm:PinSocket_2x07_P2.54mm_Vertical, B.Cu at (144.0, 39.5)
- F1, U6: moved to B.Cu
- J10: footprint Connector_PinSocket_2.54mm:PinSocket_2x07_P2.54mm_Horizontal -> Connector_PinHeader_2.54mm:PinHeader_2x07_P2.54mm_Vertical
- J11: renamed from J5; footprint Connector_Phoenix_MC:PhoenixContact_MC_1,5_12-G-3.5_1x12_P3.50mm_Horizontal -> Connector_Phoenix_MC:PhoenixContact_MC_1,5_8-G-3.5_1x08_P3.50mm_Horizontal
- J12: renamed from J6; footprint Connector_Phoenix_MC:PhoenixContact_MC_1,5_12-G-3.5_1x12_P3.50mm_Horizontal -> Connector_Phoenix_MC:PhoenixContact_MC_1,5_16-G-3.5_1x16_P3.50mm_Horizontal
- J2: renamed from J1; footprint Connector_Phoenix_MC:PhoenixContact_MC_1,5_12-G-3.5_1x12_P3.50mm_Horizontal -> Connector_Phoenix_MC:PhoenixContact_MC_1,5_16-G-3.5_1x16_P3.50mm_Horizontal
- J4: renamed from J3; footprint Connector_Phoenix_MC:PhoenixContact_MC_1,5_12-G-3.5_1x12_P3.50mm_Horizontal -> Connector_Phoenix_MC:PhoenixContact_MC_1,5_16-G-3.5_1x16_P3.50mm_Horizontal
- J8: value DI_IN_Connector -> Conn_02x07_Counter_Clockwise; footprint Connector_Phoenix_MC:PhoenixContact_MC_1,5_12-G-3.5_1x12_P3.50mm_Horizontal -> Connector_PinHeader_2.54mm:PinHeader_2x07_P2.54mm_Vertical
- J9: value Conn_01x05 -> Conn_02x07_Counter_Clockwise; footprint Connector_PinHeader_2.54mm:PinHeader_1x07_P2.54mm_Vertical -> Connector_PinHeader_2.54mm:PinHeader_2x07_P2.54mm_Vertical
- R10, R12, R13, R15, R16, R3, R4, R52, R53, R6, R7, R9: moved to F.Cu
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- renumbered J7 to J13, J13 to J16
Connections:
- C1 pad 2: Logic_GND -> LOGIC_GND
- C10 pad 2: Logic_GND -> LOGIC_GND
- C11 pad 2: Logic_GND -> LOGIC_GND
- C12 pad 2: Logic_GND -> LOGIC_GND
- C13 pad 2: Logic_GND -> LOGIC_GND
- C14 pad 2: Logic_GND -> LOGIC_GND
- C15 pad 2: Logic_GND -> LOGIC_GND
- C16 pad 2: Logic_GND -> LOGIC_GND
- C17 pad 2: Field_GND -> FIELD_GND
- C18 pad 2: Logic_GND -> LOGIC_GND
- C19 pad 2: Field_GND -> FIELD_GND
- C2 pad 2: Logic_GND -> LOGIC_GND
- C20 pad 2: Logic_GND -> LOGIC_GND
- C21 pad 2: Field_GND -> FIELD_GND
- C22 pad 2: Logic_GND -> LOGIC_GND
- C23 pad 2: Field_GND -> FIELD_GND
- C24 pad 2: Logic_GND -> LOGIC_GND
- C25 pad 2: Field_GND -> FIELD_GND
- C26 pad 2: Logic_GND -> LOGIC_GND
- C27 pad 2: Field_GND -> FIELD_GND
- C28 pad 2: Logic_GND -> LOGIC_GND
- C29 pad 2: Field_GND -> FIELD_GND
- C3 pad 2: Logic_GND -> LOGIC_GND
- C30 pad 2: Logic_GND -> LOGIC_GND
- C31 pad 2: Field_GND -> FIELD_GND
- C33 pad 2: Logic_GND -> LOGIC_GND
- C34 pad 2: Logic_GND -> LOGIC_GND
- C35 pad 2: Logic_GND -> LOGIC_GND
- C4 pad 2: Logic_GND -> LOGIC_GND
- C5 pad 2: Logic_GND -> LOGIC_GND
- C6 pad 2: Logic_GND -> LOGIC_GND
- C7 pad 2: Logic_GND -> LOGIC_GND
- C8 pad 2: Logic_GND -> LOGIC_GND
- C9 pad 2: Logic_GND -> LOGIC_GND
- CCOUT1 pad 1: 3V3_LOGIC -> +3V3
- CCOUT1 pad 2: GND -> LOGIC_GND
- CCOUT2 pad 1: 3V3_LOGIC -> +3V3
- CCOUT2 pad 2: GND -> LOGIC_GND
- CIN1 pad 2: GND -> FIELD_GND
- CIN2 pad 2: GND -> FIELD_GND
- CIN3 pad 2: GND -> FIELD_GND
- CIN4 pad 1: 5V_MAIN -> +5V
- CIN4 pad 2: GND -> LOGIC_GND
- CIN5 pad 1: 5V_MAIN -> +5V
- CIN5 pad 2: GND -> LOGIC_GND
- COUT1 pad 1: 5V_MAIN -> +5V
- COUT1 pad 2: GND -> LOGIC_GND
- COUT2 pad 1: 5V_MAIN -> +5V
- COUT2 pad 2: GND -> LOGIC_GND
- COUT3 pad 1: 5V_MAIN -> +5V
- COUT3 pad 2: GND -> LOGIC_GND
- D1 pad 2: Field_GND -> FIELD_GND
- D10 pad 2: Field_GND -> FIELD_GND
- D11 pad 2: Field_GND -> FIELD_GND
- D12 pad 2: Field_GND -> FIELD_GND
- D13 pad 2: Field_GND -> FIELD_GND
- D14 pad 2: Field_GND -> FIELD_GND
- D15 pad 2: Field_GND -> FIELD_GND
- D16 pad 2: Field_GND -> FIELD_GND
- D17 pad 2: Field_GND -> FIELD_GND
- D18 pad 2: Field_GND -> FIELD_GND
- D19 pad 2: Field_GND -> FIELD_GND
- D2 pad 2: Field_GND -> FIELD_GND
- D20 pad 2: Field_GND -> FIELD_GND
- D21 pad 2: Field_GND -> FIELD_GND
- D22 pad 2: Field_GND -> FIELD_GND
- D23 pad 2: Field_GND -> FIELD_GND
- D24 pad 2: Field_GND -> FIELD_GND
- D25 pad 2: Field_GND -> FIELD_GND
- D26 pad 2: Field_GND -> FIELD_GND
- D27 pad 1: Net-(D27-K) -> +24V
- D28 pad 1: Net-(D27-K) -> +24V
- D28 pad 2: GND -> FIELD_GND
- D29 pad 2: Field_GND -> FIELD_GND
- D3 pad 2: Field_GND -> FIELD_GND
- D30 pad 2: Field_GND -> FIELD_GND
- D4 pad 2: Field_GND -> FIELD_GND
- D5 pad 2: Field_GND -> FIELD_GND
- D6 pad 2: Field_GND -> FIELD_GND
- D7 pad 2: Field_GND -> FIELD_GND
- D8 pad 2: Field_GND -> FIELD_GND
- D9 pad 2: Field_GND -> FIELD_GND
- F1 pad 2: Net-(D27-K) -> +24V
- J10 pad 1: unconnected-(J10-Pin_1-Pad1) -> LOGIC_GND
- J10 pad 10: unconnected-(J10-Pin_10-Pad10) -> /ETH_MDIO
- J10 pad 11: unconnected-(J10-Pin_11-Pad11) -> LOGIC_GND
- J10 pad 12: unconnected-(J10-Pin_12-Pad12) -> LOGIC_GND
- J10 pad 13: unconnected-(J10-Pin_13-Pad13) -> +3V3
- J10 pad 14: unconnected-(J10-Pin_14-Pad14) -> +3V3
- J10 pad 2: unconnected-(J10-Pin_2-Pad2) -> /ETH_TXD1
- J10 pad 3: unconnected-(J10-Pin_3-Pad3) -> /ETH_TXD0
- J10 pad 4: unconnected-(J10-Pin_4-Pad4) -> /ETH_TX_EN
- J10 pad 5: unconnected-(J10-Pin_5-Pad5) -> /ETH_RXD1
- J10 pad 6: unconnected-(J10-Pin_6-Pad6) -> /ETH_RXD0
- J10 pad 7: unconnected-(J10-Pin_7-Pad7) -> /ETH_CRS_DV
- J10 pad 8: unconnected-(J10-Pin_8-Pad8) -> /ETH_REF_CLK
- J10 pad 9: unconnected-(J10-Pin_9-Pad9) -> /ETH_MDC
- J11 pad 1: +24V -> /DO_OUT14
- J11 pad 2: +24V -> /DO_OUT16
- J11 pad 3: /DO_OUT9 -> FIELD_GND
- J11 pad 4: /DO_OUT11 -> FIELD_GND
- J11 pad 5: /DO_OUT10 -> FIELD_GND
- J11 pad 6: /DO_OUT13 -> +24V
- J11 pad 7: /DO_OUT12 -> +24V
- J11 pad 8: /DO_OUT15 -> +24V
- J12 pad 1: /DI_IN4 -> /DI_IN1
- J12 pad 10: /DI_IN13 -> /DI_IN10
- J12 pad 11: /DI_IN14 -> /DI_IN11
- J12 pad 12: Field_GND -> /DI_IN12
- J12 pad 2: /DI_IN5 -> /DI_IN2
- J12 pad 3: /DI_IN6 -> /DI_IN3
- J12 pad 4: /DI_IN7 -> /DI_IN4
- J12 pad 5: /DI_IN8 -> /DI_IN5
- J12 pad 6: /DI_IN9 -> /DI_IN6
- J12 pad 7: /DI_IN10 -> /DI_IN7
- J12 pad 8: /DI_IN11 -> /DI_IN8
- J12 pad 9: /DI_IN12 -> /DI_IN9
- J16 pad 1: GND -> FIELD_GND
- J2 pad 1: unconnected-(J1-Pin_1-Pad1) -> FIELD_GND
- J2 pad 10: /DI_IN1 -> /AD7606_V5
- J2 pad 11: /DI_IN2 -> /AD7606_V4
- J2 pad 12: /DI_IN3 -> /AD7606_V3
- J2 pad 2: /AD7606_V8 -> FIELD_GND
- J2 pad 3: /AD7606_V7 -> FIELD_GND
- J2 pad 4: /AD7606_V6 -> +24V
- J2 pad 5: /AD7606_V5 -> +24V
- J2 pad 6: /AD7606_V4 -> +24V
- J2 pad 7: /AD7606_V3 -> /AD7606_V8
- J2 pad 8: /AD7606_V2 -> /AD7606_V7
- J2 pad 9: /AD7606_V1 -> /AD7606_V6
- J4 pad 11: Field_GND -> /DO_OUT9
- J4 pad 12: Field_GND -> /DO_OUT11
- J4 pad 2: +24V -> FIELD_GND
- J8 pad 1: unconnected-(J8-Pin_1-Pad1) -> +3V3
- J8 pad 10: unconnected-(J8-Pin_10-Pad10) -> LOGIC_GND
- J8 pad 11: unconnected-(J8-Pin_11-Pad11) -> +3V3
- J8 pad 12: unconnected-(J8-Pin_12-Pad12) -> LOGIC_GND
- J8 pad 2: unconnected-(J8-Pin_2-Pad2) -> LOGIC_GND
- J8 pad 3: unconnected-(J8-Pin_3-Pad3) -> +3V3
- J8 pad 4: unconnected-(J8-Pin_4-Pad4) -> LOGIC_GND
- J8 pad 5: unconnected-(J8-Pin_5-Pad5) -> +3V3
- J8 pad 6: unconnected-(J8-Pin_6-Pad6) -> LOGIC_GND
- J8 pad 7: unconnected-(J8-Pin_7-Pad7) -> +3V3
- J8 pad 8: unconnected-(J8-Pin_8-Pad8) -> LOGIC_GND
- J8 pad 9: unconnected-(J8-Pin_9-Pad9) -> +3V3
- J9 pad 1: /MCU_STM32/DAC8568_SCLK -> +5V
- J9 pad 2: /MCU_STM32/DAC8568_DIN -> LOGIC_GND
- J9 pad 3: /MCU_STM32/DAC8568_CLR -> +5V
- J9 pad 4: /MCU_STM32/DAC8568_SYNC -> LOGIC_GND
- J9 pad 5: /MCU_STM32/DAC8568_LDAC -> +5V
- J9 pad 6: Logic_GND -> LOGIC_GND
- L1 pad 2: 5V_MAIN -> +5V
- MOD1 pad 1: Logic_GND -> LOGIC_GND
- MOD1 pad 2: unconnected-(MOD1-+5V-Pad2) -> +5V
- MOD1 pad 43: unconnected-(MOD1-B13-Pad43) -> /MCU_STM32/ETH_TXD1
- MOD1 pad 44: unconnected-(MOD1-B12-Pad44) -> /MCU_STM32/ETH_TXD0
- MOD1 pad 45: Logic_GND -> LOGIC_GND
- MOD1 pad 46: unconnected-(MOD1-+3V3-Pad46) -> +3V3
- MOD1 pad 56: unconnected-(MOD1-C1-Pad56) -> /MCU_STM32/ETH_MDC
- MOD1 pad 59: Logic_GND -> LOGIC_GND
- MOD1 pad 62: unconnected-(MOD1-A1-Pad62) -> /MCU_STM32/ETH_REF_CLK
- MOD1 pad 63: unconnected-(MOD1-A2-Pad63) -> /MCU_STM32/ETH_MDIO
- MOD1 pad 68: unconnected-(MOD1-A7-Pad68) -> /MCU_STM32/ETH_CRS_DV
- MOD1 pad 69: unconnected-(MOD1-C4-Pad69) -> /MCU_STM32/ETH_RXD0
- MOD1 pad 70: unconnected-(MOD1-C5-Pad70) -> /MCU_STM32/ETH_RXD1
- MOD1 pad 84: unconnected-(MOD1-B11-Pad84) -> /MCU_STM32/ETH_TX_EN
- MOD1 pad 85: unconnected-(MOD1-3V3-Pad85) -> +3V3
- MOD1 pad 86: unconnected-(MOD1-5V-Pad86) -> +5V
- MOD1 pad 87: Logic_GND -> LOGIC_GND
- MOD1 pad 88: Logic_GND -> LOGIC_GND
- Q2 pad 2: Net-(D27-K) -> +24V
- R50 pad 2: GND -> FIELD_GND
- R51 pad 2: Net-(D27-K) -> +24V
- RFBB1 pad 2: GND -> LOGIC_GND
- RFBB1_TRIM1 pad 2: GND -> LOGIC_GND
- RFBT1 pad 1: 5V_MAIN -> +5V
- RFBT1_TRIM1 pad 1: 5V_MAIN -> +5V
- U1 pad 1: Logic_GND -> LOGIC_GND
- U1 pad 3: Logic_GND -> LOGIC_GND
- U1 pad 32: Logic_GND -> FIELD_GND
- U1 pad 34: Logic_GND -> FIELD_GND
- U1 pad 36: Logic_GND -> FIELD_GND
- U1 pad 38: Logic_GND -> FIELD_GND
- U1 pad 4: Logic_GND -> LOGIC_GND
- U1 pad 40: Logic_GND -> FIELD_GND
- U1 pad 42: Logic_GND -> FIELD_GND
- U1 pad 44: Logic_GND -> FIELD_GND
- U1 pad 46: Logic_GND -> FIELD_GND
- U1 pad 5: Logic_GND -> LOGIC_GND
- U10 pad 3: Field_GND -> FIELD_GND
- U10 pad 5: Logic_GND -> LOGIC_GND
- U11 pad 3: Logic_GND -> LOGIC_GND
- U12 pad 3: Field_GND -> FIELD_GND
- U12 pad 5: Logic_GND -> LOGIC_GND
- U13 pad 3: Logic_GND -> LOGIC_GND
- U14 pad 2: Field_GND -> FIELD_GND
- U14 pad 3: Logic_GND -> LOGIC_GND
- U15 pad 3: Logic_GND -> LOGIC_GND
- U16 pad 2: Field_GND -> FIELD_GND
- U16 pad 3: Logic_GND -> LOGIC_GND
- U17 pad 3: Logic_GND -> LOGIC_GND
- U18 pad 2: Field_GND -> FIELD_GND
- U18 pad 3: Logic_GND -> LOGIC_GND
- U19 pad 3: Logic_GND -> LOGIC_GND
- U2 pad 3: Logic_GND -> LOGIC_GND
- U20 pad 2: Field_GND -> FIELD_GND
- U20 pad 3: Logic_GND -> LOGIC_GND
- U21 pad 3: Logic_GND -> LOGIC_GND
- U22 pad 2: Field_GND -> FIELD_GND
- U22 pad 3: Logic_GND -> LOGIC_GND
- U23 pad 3: Logic_GND -> LOGIC_GND
- U24 pad 2: Field_GND -> FIELD_GND
- U24 pad 3: Logic_GND -> LOGIC_GND
- U25 pad 3: Logic_GND -> LOGIC_GND
- U26 pad 2: Field_GND -> FIELD_GND
- U26 pad 3: Logic_GND -> LOGIC_GND
- U27 pad 3: Logic_GND -> LOGIC_GND
- U28 pad 2: Field_GND -> FIELD_GND
- U28 pad 3: Logic_GND -> LOGIC_GND
- U29 pad 1: GND -> FIELD_GND
- U3 pad 3: Field_GND -> FIELD_GND
- U3 pad 5: Logic_GND -> LOGIC_GND
- U30 pad 1: 5V_MAIN -> +5V
- U30 pad 2: GND -> LOGIC_GND
- U30 pad 3: 3V3_LOGIC -> +3V3
- U31 pad 3: Logic_GND -> LOGIC_GND
- U32 pad 3: Field_GND -> FIELD_GND
- U32 pad 5: Logic_GND -> LOGIC_GND
- U4 pad 3: Logic_GND -> LOGIC_GND
- U5 pad 3: Field_GND -> FIELD_GND
- U5 pad 5: Logic_GND -> LOGIC_GND
- U6 pad 1: Logic_GND -> LOGIC_GND
- U7 pad 3: Logic_GND -> LOGIC_GND
- U8 pad 3: Field_GND -> FIELD_GND
- U8 pad 5: Logic_GND -> LOGIC_GND
- U9 pad 3: Logic_GND -> LOGIC_GND
Routing:
- net +5V: track 140.0 -> 949.7 mm, vias 0 -> 15
- net +3V3: track 151.7 -> 656.9 mm, vias 8 -> 13
- net LOGIC_GND: track 0.00 -> 271.0 mm, vias 0 -> 218
- net /MCU_STM32/ETH_RXD0: track 0.00 -> 200.5 mm, vias 0 -> 1
- net /MCU_STM32/ETH_RXD1: track 0.00 -> 191.2 mm, vias 0 -> 1
- net /MCU_STM32/ETH_CRS_DV: track 0.00 -> 174.3 mm, vias 0 -> 1
- net /MCU_STM32/ETH_MDIO: track 0.00 -> 135.2 mm, vias 0 -> 2
- net /MCU_STM32/ETH_MDC: track 0.00 -> 128.1 mm, vias 0 -> 1
- net /MCU_STM32/ETH_REF_CLK: track 0.00 -> 103.9 mm, vias 0 -> 1
- net /MCU_STM32/ETH_TXD1: track 0.00 -> 89.6 mm, vias 0 -> 1
- net /MCU_STM32/ETH_TXD0: track 0.00 -> 87.7 mm, vias 0 -> 1
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- added copper zone on B.Cu, net +24V
- added copper zone on F.Cu, net +24V
- added copper zone on B.Cu, net FIELD_GND
- added copper zone on F.Cu, net FIELD_GND
- added copper zone on B.Cu, net LOGIC_GND
- added copper zone on F.Cu, net LOGIC_GND
Other:
- board size 175.3 x 163.3 mm -> 151 x 158.2 mm
