File: .history/MY_POWERFULL_PLC_PCB.kicad_pcb (KiCad board)
At the start: 2 copper layers, 151 x 158.2 mm, 287 parts, among them J1 DI_IN_Connector, J10 Conn_02x07_Counter_Clockwise, J11 DI_IN_Connector, J12 DI_IN_Connector, J13 DI_IN_Connector, J14 Conn_02x20_Counter_Clockwise, J15 Conn_02x07_Counter_Clockwise, J16 DI_IN_Connector, J2 DI_IN_Connector, J3 Conn_02x20_Counter_Clockwise, J4 DI_IN_Connector, J5 Conn_02x07_Counter_Clockwise, J6 Conn_02x07_Counter_Clockwise, J7 Conn_02x07_Counter_Clockwise, J8 Conn_02x07_Counter_Clockwise, J9 Conn_02x07_Counter_Clockwise, Q1 NMOS AOD4184A, Q10 NMOS AOD4184A, Q11 NMOS AOD4184A, Q12 NMOS AOD4184A, Q13 NMOS AOD4184A, Q14 NMOS AOD4184A, Q15 NMOS AOD4184A, Q16 NMOS AOD4184A, Q17 NMOS AOD4184A, Q2 Q_PMOS, Q3 NMOS AOD4184A, Q4 NMOS AOD4184A, Q5 NMOS AOD4184A, Q6 NMOS AOD4184A, Q7 NMOS AOD4184A, Q8 NMOS AOD4184A, Q9 NMOS AOD4184A, U10 6N137, U11 SN74LVC1G17DBVR, U12 6N137, U13 SN74LVC1G14DBV, U14 LTV-357T, U15 SN74LVC1G14DBV, U16 LTV-357T, U17 SN74LVC1G14DBV, U18 LTV-357T, U19 SN74LVC1G14DBV, U2 SN74LVC1G17DBVR, U20 LTV-357T, U21 SN74LVC1G14DBV, U22 LTV-357T, U23 SN74LVC1G14DBV, U24 LTV-357T, U25 SN74LVC1G14DBV, U26 LTV-357T, U27 SN74LVC1G14DBV, U28 LTV-357T, U29 LMR51430, U3 6N137, U30 AP7361C-33E, U31 SN74LVC1G17DBVR, U32 6N137, U33 UCC27511ADBV, U34 UCC27511ADBV, U35 UCC27511ADBV, U36 UCC27511ADBV, U37 UCC27511ADBV, U38 UCC27511ADBV, U39 UCC27511ADBV, U4 SN74LVC1G17DBVR, U40 UCC27511ADBV, U5 6N137, U7 SN74LVC1G17DBVR, U8 6N137, U9 SN74LVC1G17DBVR

Commit message: 112
Parts:
- removed the J13 at (200.9, 200.2)
- removed the J6 at (144.0, 32.3)
- removed the J7 at (144.0, 39.5)
- added J11: Conn_02x07_Counter_Clockwise, Connector_PinSocket_2.54mm:PinSocket_2x07_P2.54mm_Vertical, F.Cu at (159.1, 32.3)
- added J12: Conn_02x07_Counter_Clockwise, Connector_PinSocket_2.54mm:PinSocket_2x07_P2.54mm_Vertical, F.Cu at (159.1, 39.5)
- moved D44 21.0 mm to (108.4, 165.6)
- moved D46 21.0 mm to (112.0, 165.6)
- moved D42 19.4 mm to (97.9, 165.6)
- moved R90 18.6 mm to (115.7, 141.0)
- moved R91 18.6 mm to (115.7, 138.7)
- moved R92 18.6 mm to (115.7, 143.3)
- moved C46 17.4 mm to (110.1, 141.9)
- moved C47 17.4 mm to (110.1, 143.9)
- moved U38 17.4 mm to (109.7, 139.2)
- moved R89 17.4 mm to (106.6, 136.0)
- moved Q15 17.4 mm to (111.4, 152.3)
- moved R97 15.1 mm to (114.0, 134.4)
- moved C50 15.0 mm to (113.5, 141.2)
- moved C51 15.0 mm to (113.5, 143.2)
- moved Q17 15.0 mm to (110.0, 151.3)
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- renumbered J12 to J10, J14 to J13, J15 to J14, J16 to J15, J11 to J5, J5 to J6, J8 to J7, J9 to J8, J10 to J9
Connections:
- C1 pad 2: LOGIC_GND -> FIELD_GND
- C10 pad 2: LOGIC_GND -> FIELD_GND
- C11 pad 2: LOGIC_GND -> FIELD_GND
- C12 pad 2: LOGIC_GND -> FIELD_GND
- C13 pad 2: LOGIC_GND -> FIELD_GND
- C14 pad 2: LOGIC_GND -> FIELD_GND
- C15 pad 2: LOGIC_GND -> FIELD_GND
- C16 pad 2: LOGIC_GND -> FIELD_GND
- C18 pad 2: LOGIC_GND -> FIELD_GND
- C2 pad 2: LOGIC_GND -> FIELD_GND
- C20 pad 2: LOGIC_GND -> FIELD_GND
- C22 pad 2: LOGIC_GND -> FIELD_GND
- C24 pad 2: LOGIC_GND -> FIELD_GND
- C26 pad 2: LOGIC_GND -> FIELD_GND
- C28 pad 2: LOGIC_GND -> FIELD_GND
- C3 pad 2: LOGIC_GND -> FIELD_GND
- C30 pad 2: LOGIC_GND -> FIELD_GND
- C33 pad 2: LOGIC_GND -> FIELD_GND
- C34 pad 2: LOGIC_GND -> FIELD_GND
- C35 pad 2: LOGIC_GND -> FIELD_GND
- C4 pad 2: LOGIC_GND -> FIELD_GND
- C5 pad 2: LOGIC_GND -> FIELD_GND
- C6 pad 2: LOGIC_GND -> FIELD_GND
- C7 pad 2: LOGIC_GND -> FIELD_GND
- C8 pad 2: LOGIC_GND -> FIELD_GND
- C9 pad 2: LOGIC_GND -> FIELD_GND
- CCOUT1 pad 2: LOGIC_GND -> FIELD_GND
- CCOUT2 pad 2: LOGIC_GND -> FIELD_GND
- CIN4 pad 2: LOGIC_GND -> FIELD_GND
- CIN5 pad 2: LOGIC_GND -> FIELD_GND
- COUT1 pad 2: LOGIC_GND -> FIELD_GND
- COUT2 pad 2: LOGIC_GND -> FIELD_GND
- COUT3 pad 2: LOGIC_GND -> FIELD_GND
- J13 pad 1: +5V -> +5V_Core
- J13 pad 2: +3V3 -> +3V3_Core
- J13 pad 21: LOGIC_GND -> GND_Core
- J13 pad 22: LOGIC_GND -> GND_Core
- J13 pad 23: LOGIC_GND -> GND_Core
- J13 pad 24: LOGIC_GND -> GND_Core
- J13 pad 25: LOGIC_GND -> GND_Core
- J13 pad 26: LOGIC_GND -> GND_Core
- J13 pad 27: +5V -> +5V_Core
- J13 pad 28: +5V -> +5V_Core
- J13 pad 3: LOGIC_GND -> GND_Core
- J13 pad 4: LOGIC_GND -> GND_Core
- J13 pad 45: LOGIC_GND -> GND_Core
- J13 pad 46: LOGIC_GND -> GND_Core
- J13 pad 47: +3V3 -> +3V3_Core
- J13 pad 48: +3V3 -> +3V3_Core
- J13 pad 5: LOGIC_GND -> GND_Core
- J13 pad 7: LOGIC_GND -> GND_Core
- J14 pad 1: LOGIC_GND -> GND_Core
- J14 pad 11: LOGIC_GND -> GND_Core
- J14 pad 12: LOGIC_GND -> GND_Core
- J14 pad 13: +3V3 -> +3V3_Core
- J14 pad 14: +3V3 -> +3V3_Core
- J3 pad 1: unconnected-(J3-Pin_1-Pad1) -> FIELD_GND
- J3 pad 2: unconnected-(J3-Pin_2-Pad2) -> +5V
- J3 pad 21: LOGIC_GND -> FIELD_GND
- J3 pad 22: LOGIC_GND -> FIELD_GND
- J3 pad 23: LOGIC_GND -> FIELD_GND
- J3 pad 24: LOGIC_GND -> FIELD_GND
- J3 pad 25: LOGIC_GND -> FIELD_GND
- J3 pad 26: LOGIC_GND -> FIELD_GND
- J3 pad 3: unconnected-(J3-Pin_3-Pad3) -> FIELD_GND
- J3 pad 31: /DO_PWM_CTRL2 -> /DO_PWM_CTRL3
- J3 pad 33: /DO_PWM_CTRL3 -> /DO_PWM_CTRL2
- J3 pad 35: /DO_PWM_CTRL4 -> /DO_PWM_CTRL5
- J3 pad 37: /DO_PWM_CTRL5 -> /DO_PWM_CTRL4
- J3 pad 39: /DO_PWM_CTRL6 -> /DO_PWM_CTRL7
- J3 pad 4: unconnected-(J3-Pin_4-Pad4) -> +3V3
- J3 pad 41: /DO_PWM_CTRL7 -> /DO_PWM_CTRL6
- J3 pad 45: LOGIC_GND -> FIELD_GND
- J3 pad 46: LOGIC_GND -> FIELD_GND
- J3 pad 55: unconnected-(J3-Pin_55-Pad55) -> +5V
- J3 pad 56: unconnected-(J3-Pin_56-Pad56) -> FIELD_GND
- J3 pad 6: LOGIC_GND -> FIELD_GND
- J3 pad 8: LOGIC_GND -> FIELD_GND
- J4 pad 13: /DO_OUT10 -> unconnected-(J4-Pin_13-Pad13)
- J4 pad 14: /DO_OUT13 -> unconnected-(J4-Pin_14-Pad14)
- J4 pad 15: /DO_OUT12 -> /DO_OUT13
- J4 pad 16: /DO_OUT15 -> /DO_OUT10
- J5 pad 1: /DO_OUT14 -> unconnected-(J5-Pin_1-Pad1)
- J5 pad 2: /DO_OUT16 -> unconnected-(J5-Pin_2-Pad2)
- J5 pad 3: FIELD_GND -> /DO_OUT15
- J5 pad 4: FIELD_GND -> /DO_OUT12
- J5 pad 5: FIELD_GND -> unconnected-(J5-Pin_5-Pad5)
- J5 pad 6: +24V -> unconnected-(J5-Pin_6-Pad6)
- J5 pad 7: +24V -> /DO_OUT14
- J5 pad 8: +24V -> /DO_OUT16
- J6 pad 1: LOGIC_GND -> FIELD_GND
- J6 pad 11: LOGIC_GND -> FIELD_GND
- J6 pad 12: LOGIC_GND -> FIELD_GND
- J7 pad 10: LOGIC_GND -> FIELD_GND
- J7 pad 12: LOGIC_GND -> FIELD_GND
- J7 pad 14: LOGIC_GND -> FIELD_GND
- J7 pad 2: LOGIC_GND -> FIELD_GND
- J7 pad 4: LOGIC_GND -> FIELD_GND
- J7 pad 6: LOGIC_GND -> FIELD_GND
- J7 pad 8: LOGIC_GND -> FIELD_GND
- J8 pad 10: LOGIC_GND -> FIELD_GND
- J8 pad 11: +5V -> FIELD_GND
- J8 pad 12: LOGIC_GND -> FIELD_GND
- J8 pad 13: +5V -> FIELD_GND
- J8 pad 14: LOGIC_GND -> FIELD_GND
- J8 pad 2: LOGIC_GND -> FIELD_GND
- J8 pad 4: LOGIC_GND -> FIELD_GND
- J8 pad 6: LOGIC_GND -> FIELD_GND
- J8 pad 8: LOGIC_GND -> FIELD_GND
- J9 pad 1: LOGIC_GND -> FIELD_GND
- J9 pad 11: LOGIC_GND -> FIELD_GND
- J9 pad 12: LOGIC_GND -> FIELD_GND
- MOD1 pad 1: LOGIC_GND -> GND_Core
- MOD1 pad 2: +5V -> +5V_Core
- MOD1 pad 45: LOGIC_GND -> GND_Core
- MOD1 pad 46: +3V3 -> +3V3_Core
- MOD1 pad 59: LOGIC_GND -> GND_Core
- MOD1 pad 85: +3V3 -> +3V3_Core
- MOD1 pad 86: +5V -> +5V_Core
- MOD1 pad 87: LOGIC_GND -> GND_Core
- MOD1 pad 88: LOGIC_GND -> GND_Core
- RFBB1 pad 2: LOGIC_GND -> FIELD_GND
- RFBB1_TRIM1 pad 2: LOGIC_GND -> FIELD_GND
- U1 pad 1: LOGIC_GND -> FIELD_GND
- U1 pad 3: LOGIC_GND -> FIELD_GND
- U1 pad 4: LOGIC_GND -> FIELD_GND
- U1 pad 5: LOGIC_GND -> FIELD_GND
- U10 pad 5: LOGIC_GND -> FIELD_GND
- U11 pad 3: LOGIC_GND -> FIELD_GND
- U12 pad 5: LOGIC_GND -> FIELD_GND
- U13 pad 3: LOGIC_GND -> FIELD_GND
- U14 pad 3: LOGIC_GND -> FIELD_GND
- U15 pad 3: LOGIC_GND -> FIELD_GND
- U16 pad 3: LOGIC_GND -> FIELD_GND
- U17 pad 3: LOGIC_GND -> FIELD_GND
- U18 pad 3: LOGIC_GND -> FIELD_GND
- U19 pad 3: LOGIC_GND -> FIELD_GND
- U2 pad 3: LOGIC_GND -> FIELD_GND
- U20 pad 3: LOGIC_GND -> FIELD_GND
- U21 pad 3: LOGIC_GND -> FIELD_GND
- U22 pad 3: LOGIC_GND -> FIELD_GND
- U23 pad 3: LOGIC_GND -> FIELD_GND
- U24 pad 3: LOGIC_GND -> FIELD_GND
- U25 pad 3: LOGIC_GND -> FIELD_GND
- U26 pad 3: LOGIC_GND -> FIELD_GND
- U27 pad 3: LOGIC_GND -> FIELD_GND
- U28 pad 3: LOGIC_GND -> FIELD_GND
- U3 pad 5: LOGIC_GND -> FIELD_GND
- U30 pad 2: LOGIC_GND -> FIELD_GND
- U31 pad 3: LOGIC_GND -> FIELD_GND
- U32 pad 5: LOGIC_GND -> FIELD_GND
- U4 pad 3: LOGIC_GND -> FIELD_GND
- U5 pad 5: LOGIC_GND -> FIELD_GND
- U6 pad 1: LOGIC_GND -> GND_Core
- U6 pad 2: +5V -> +5V_Core
- U7 pad 3: LOGIC_GND -> FIELD_GND
- U8 pad 5: LOGIC_GND -> FIELD_GND
- U9 pad 3: LOGIC_GND -> FIELD_GND
Routing:
- net +24V: track 30.6 -> 608.2 mm, vias 0 -> 18
- net +3V3_Core: track 0.00 -> 398.1 mm, vias 0 -> 4
- net FIELD_GND: track 2.30 -> 357.4 mm, vias 38 -> 333
- net +5V: track 949.7 -> 622.2 mm, vias 15 -> 22
- net LOGIC_GND: track 271.0 -> 0.00 mm, vias 218 -> 0
- net +5V_Core: track 0.00 -> 266.0 mm, vias 0 -> 5
- net +3V3: track 656.9 -> 412.1 mm, vias 13 -> 8
- net GND_Core: track 0.00 -> 33.0 mm, vias 0 -> 209
- net /DO_PWM_CTRL8: track 27.8 -> 43.2 mm
- net /DO_PWM_CTRL6: track 22.8 -> 38.1 mm, vias 0 -> 1
- net /DO_OUT14: track 22.8 -> 8.69 mm
- net /DO_PWM_CTRL7: track 19.0 -> 32.2 mm
- net /DO_OUT16: track 21.8 -> 9.24 mm
- net /DO_OUT12: track 20.0 -> 7.76 mm
- net /DO_OUT10: track 19.0 -> 7.86 mm
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- added copper zone on B.Cu, net GND_Core
- added copper zone on F.Cu, net GND_Core
- removed copper zone on B.Cu, net +24V
- removed copper zone on F.Cu, net +24V
- removed copper zone on B.Cu, net LOGIC_GND
- removed copper zone on F.Cu, net LOGIC_GND

Commit message: 112
Routing:
- net FIELD_GND: vias 333 -> 334
Changed lines of the file:
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@@
 			(drillshape 0)
 			(scaleselection 1)
-			(outputdirectory "./")
+			(outputdirectory "Gerber/")
 		)
 	)
@@
 	)
 	(via
+		(at 78.649413 108.574413)
+		(size 0.6)
+		(drill 0.3)
+		(layers "F.Cu" "B.Cu")
+		(net "FIELD_GND")
+	)
+	(via
 		(at 63 155)
 		(size 0.6)
@@
 		(polygon
 			(pts
-				(xy 5.528437 135.155875) (xy 5.596752 172.17164) (xy 175.045527 171.800682) (xy 174.964638 134.843216)
-			)
-		)
-	)
-	(zone
-		(net "FIELD_GND")
-		(layers "F.Cu" "B.Cu")
-		(hatch edge 0.5)
-		(priority 2)
-		(connect_pads yes
-			(clearance 0.5)
-		)
-		(min_thickness 0.5)
-		(fill yes
-			(thermal_gap 0.5)
-			(thermal_bridge_width 0.5)
-			(island_removal_mode 0)
-		)
-		(polygon
-			(pts
-				(xy 5.570065 83.426356) (xy 5.617362 108.999078) (xy 175.071467 108.62815) (xy 175.015727 83.113633)
-			)
-		)
-	)
-	(zone
-		(net "FIELD_GND")
-		(layers "F.Cu" "B.Cu")
-		(hatch edge 0.5)
-		(priority 2)
-		(connect_pads yes
-			(clearance 0.5)
-		)
-		(min_thickness 0.5)
-		(fill yes
-			(thermal_gap 0.5)
-			(thermal_bridge_width 0.5)
-			(island_removal_mode 0)
-		)
-		(polygon
-			(pts
-				(xy 5.54173 109.116354) (xy 5.589275 134.815474) (xy 175.043387 134.444544) (xy 174.987385 108.80363)
+				(xy 5.435034 84.546306) (xy 5.596752 172.17164) (xy 175.045527 171.800682) (xy 174.853869 84.233678)
 			)
 		)
